File: greenenergyecu.kicad_pcb (KiCad board)
At the start: 2 copper layers, 272 x 194 mm, 0 parts

Commit message: version 8
Other:
- board size 272 x 194 mm -> 272 x 183 mm
Changed lines of the file:
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@@
 		(layer "Edge.Cuts")
 	)
-	(gr_rect
-		(start 165.5 98)
-		(end 170.5 129.5)
+	(gr_line
+		(start 215.5 129)
+		(end 67 127.5)
 		(stroke
 			(width 0.05)
 			(type default)
 		)
-		(fill none)
 		(layer "Edge.Cuts")
 	)
-	(gr_rect
-		(start 37 3)
-		(end 284 197)
+	(gr_line
+		(start 67 127.5)
+		(end 42.5 25)
 		(stroke
 			(width 0.05)
 			(type default)
 		)
-		(fill none)
+		(layer "Edge.Cuts")
+	)
+	(gr_line
+		(start 42.5 25)
+		(end 226 26)
+		(stroke
+			(width 0.05)
+			(type default)
+		)
 		(layer "Edge.Cuts")
 	)
@@
 		(layer "Edge.Cuts")
 	)
-	(gr_rect
-		(start 85.5 65.5)
-		(end 132 127.5)
+	(gr_line
+		(start 226 26)
+		(end 215.5 129)
 		(stroke
 			(width 0.05)
 			(type default)
 		)
-		(fill none)
 		(layer "Edge.Cuts")
 	)

Commit message: version 8
Parts:
- added U1: ICM7555xB, Package_SO:SOIC-8_3.9x4.9mm_P1.27mm, F.Cu at (122.0, 69.0)
Routing:
- net Net-(U1-GND): track 0.00 -> 1.27 mm
Other:
- outline, holes or cut-outs redrawn

Commit message: version 8
Other:
- board size 272 x 183 mm -> 17.5 x 11.5 mm
Changed lines of the file:
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@@
 		)
-	)
-	(gr_rect
-		(start 12.5 14)
-		(end 284.5 14)
-		(stroke
-			(width 0.05)
-			(type default)
-		)
-		(fill none)
-		(layer "Edge.Cuts")
 	)
 	(gr_poly
 		(pts
-			(xy 121.5 74.5) (xy 131 75.5) (xy 129.5 64) (xy 114.5 63.5) (xy 108.5 63.5) (xy 122 77)
+			(xy 129.5 74.5) (xy 128.5 63) (xy 115.5 63.5) (xy 112 74)
 		)
 		(stroke
@@
 		)
 		(fill none)
-		(layer "Edge.Cuts")
-	)
-	(gr_rect
-		(start 283.5 14)
-		(end 284.5 197)
-		(stroke
-			(width 0.05)
-			(type default)
-		)
-		(fill none)

Commit message: rt
Parts:
- removed U1: ICM7555xB, Package_SO:SOIC-8_3.9x4.9mm_P1.27mm
- added M1: Module-knock-0.2, hellen-one-knock-0.2:knock, F.Cu at (116.5, 69.2)
Routing:
- net Net-(U1-GND): track 1.27 -> 0.00 mm

Commit message: err
Other:
- board size 17.5 x 11.5 mm -> 10.5 x 7.5 mm
Changed lines of the file:
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@@
 		(pad_to_mask_clearance 0)
 		(allow_soldermask_bridges_in_footprints no)
-		(aux_axis_origin 119 64)
+		(aux_axis_origin 116 63.5)
+		(grid_origin 116 63.5)
 		(pcbplotparams
 			(layerselection 0x00010fc_ffffffff)
@@
 		)
 	)
-	(gr_poly
-		(pts
-			(xy 129.5 74.5) (xy 128.5 63) (xy 115.5 63.5) (xy 112 74)
-		)
+	(gr_rect
+		(start 116 63.5)
+		(end 126.5 71)
 		(stroke
 			(width 0.05)
-			(type solid)
+			(type default)
 		)
 		(fill none)

Commit message: ee
Parts:
- added REF**: M600, 0.5:wbo, F.Cu at (120.0, 65.0)
Other:
- board size 10.5 x 7.5 mm -> 33.5 x 23.5 mm
