File: greenenergyecu.kicad_pcb (KiCad board)
At the start: 4 copper layers, 164 x 118 mm, 103 parts, among them J21 Conn_01x05_Male, J22 USB_B_Mini, M1 Module-power_12and5V-0.3, M2 Module-knock-0.2, M3 Module-vr-discrete-0.5, M4 Module-vr-max9924-0.1, M5 Module-wbo-0.5, M6 Module:mega-mcu100/0.3, M7 Module-can-0.1, M8 Module-motor-driver-0.1, P1 368255-2, Q1 ISL9V3040D3ST, Q2 ISL9V3040D3ST, Q3 ISL9V3040D3ST, Q4 ISL9V3040D3ST, Q5 ISL9V3040D3ST, Q6 ISL9V3040D3ST, Q7 AO3400A, U1 VNLD5160TR-E, U10 BTS6143D, U2 VNLD5160TR-E, U3 VNLD5160TR-E, U4 VNLD5160TR-E, U5 VNLD5160TR-E, U6 VNLD5160TR-E, U7 VNLD5160TR-E, U8 MAX31855KASA

Commit message: weW
Parts:
- added G4: DISCLAIMER, rusefi_lib:Off_Road_Disclaimer, B.Cu at (111.8, 0.28)
- P1: footprint 368255-2:368255-2 -> hellen121vag:368255-2
- moved P1 139.4 mm to (60.2, 32.9), turned to 0 degrees
- moved R22 95.2 mm to (161.9, 33.9)
- moved R23 95.2 mm to (161.9, 35.8)
- moved R24 95.2 mm to (161.9, 37.8)
- moved R28 95.2 mm to (161.9, 39.7)
- moved R29 95.2 mm to (161.9, 41.7)
- moved R30 95.2 mm to (161.9, 43.6)
- moved R46 95.0 mm to (160.8, 55.7)
- moved R47 95.0 mm to (160.8, 57.7)
- moved R48 95.0 mm to (160.8, 59.6)
- moved R49 95.0 mm to (160.8, 61.6)
- moved R34 95.0 mm to (154.2, 55.7)
- moved R35 95.0 mm to (154.2, 57.7)
- moved R36 95.0 mm to (154.2, 59.6)
- moved R37 95.0 mm to (154.2, 61.6)
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Routing:
- net PIN2: vias 0 -> 31
- net PIN113: vias 30 -> 0
- added copper zone on B.Cu, net PIN2
- added copper zone on F.Cu, net PIN2
- added copper zone on In1.Cu, net PIN2
- removed copper zone on B.Cu, net PIN113
- removed copper zone on F.Cu, net PIN113
Other:
- outline, holes or cut-outs redrawn
- board text added: "1"
- board text added: "10"
- board text added: "100"
- board text added: "101"
- board text added: "102"
- board text added: "103"
- board text added: "104"
- board text added: "105"
- board text added: "106"
- board text added: "11"
- board text added: "112"
- board text added: "113"
- board text added: "114"
- board text added: "115"
- board text added: "116"
- board text added: "117"
- board text added: "118"
- board text added: "119"
- board text added: "12"
- board text added: "120"
- board text added: "121"
- board text added: "13"
- board text added: "14"
- board text added: "15"
- board text added: "16"
- board text added: "17"
- board text added: "18"
- board text added: "19"
- board text added: "2"
- board text added: "20"
- board text added: "21"
- board text added: "22"
- board text added: "23"
- board text added: "24"
- board text added: "25"
- board text added: "26"
- board text added: "27"
- board text added: "28"
- board text added: "29"
- board text added: "3"
- board text added: "30"
- board text added: "31"
- board text added: "32"
- board text added: "33"
- board text added: "34"
- board text added: "35"
- board text added: "36"
- board text added: "37"
- board text added: "38"
- board text added: "39"
- board text added: "4"
- board text added: "40"
- board text added: "41"
- board text added: "42"
- board text added: "43"
- board text added: "44"
- board text added: "45"
- board text added: "46"
- board text added: "47"
- board text added: "48"
- board text added: "49"
- board text added: "5"
- board text added: "50"
- board text added: "51"
- board text added: "52"
- board text added: "53"
- board text added: "54"
- board text added: "55"
- board text added: "56"
- board text added: "57"
- board text added: "58"
- board text added: "59"
- board text added: "6"
- board text added: "60"
- board text added: "61"
- board text added: "62"
- board text added: "63"
- board text added: "64"
- board text added: "65"
- board text added: "66"
- board text added: "67"
- board text added: "68"
- board text added: "69"
- board text added: "7"
- board text added: "70"
- board text added: "71"
- board text added: "72"
- board text added: "73"
- board text added: "74"
- board text added: "75"
- board text added: "76"
- board text added: "77"
- board text added: "78"
- board text added: "79"
- board text added: "8"
- board text added: "80"
- board text added: "81"
- board text added: "82"
- board text added: "83"
- board text added: "84"
- board text added: "85"
- board text added: "86"
- board text added: "87"
- board text added: "88"
- board text added: "89"
- board text added: "9"
- board text added: "90"
- board text added: "91"
- board text added: "92"
- board text added: "93"
- board text added: "94"
- board text added: "95"
- board text added: "96"
- board text added: "97"
- board text added: "98"
- board text added: "99"

Commit message: weW
Parts:
- removed G4: DISCLAIMER, rusefi_lib:Off_Road_Disclaimer
Changed lines of the file:
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@@
 		)
-	)
-	(footprint "rusefi_lib:Off_Road_Disclaimer"
-		(locked yes)
-		(layer "B.Cu")
-		(at 111.75 0.275 180)
-		(property "Reference" "G4"
-			(at 0 5.715 0)
-			(layer "B.SilkS")
-			(hide yes)
-			(effects
-				(font
-					(size 1.524 1.524)
-					(thickness 0.3048)
-				)
-				(justify mirror)
-			)
-		)
-		(property "Value" "DISCLAIMER"
-			(at 0 8.255 0)
-			(layer "B.SilkS")
-			(hide yes)
-			(effects
-				(font
-					(size 1.524 1.524)
-					(thickness 0.3048)
-				)
-				(justify mirror)
-			)
-		)
-		(property "Footprint" ""
-			(at 0 0 180)
-			(layer "F.Fab")
-			(hide yes)
-			(effects
-				(font
-					(size 1.27 1.27)
-					(thickness 0.15)
-				)
-			)
-		)
-		(property "Datasheet" ""
-			(at 0 0 180)
-			(layer "F.Fab")
-			(hide yes)
-			(effects
-				(font
-					(size 1.27 1.27)
-					(thickness 0.15)
-				)
-			)
-		)
-		(property "Description" ""
-			(at 0 0 180)
-			(layer "F.Fab")
-			(hide yes)
-			(effects
-				(font
-					(size 1.27 1.27)
-					(thickness 0.15)
-				)
-			)
-		)
-		(sheetfile "hellen121vag.kicad_sch")
-		(attr through_hole)
 	)
 	(gr_line
@@
 		(min_thickness 0.254)
 		(filled_areas_thickness no)
-		(fill
+		(fill yes
 			(thermal_gap 0.508)
 			(thermal_bridge_width 0.508)
@@
 		(min_thickness 0.2)
 		(filled_areas_thickness no)
-		(fill
+		(fill yes
 			(thermal_gap 0.2)
 			(thermal_bridge_width 0.5)
@@
 		(min_thickness 0.254)
 		(filled_areas_thickness no)
-		(fill
+		(fill yes
 			(thermal_gap 0.508)
 			(thermal_bridge_width 0.508)
@@
 		(min_thickness 0.2)
 		(filled_areas_thickness no)
-		(fill
+		(fill yes
 			(thermal_gap 0.2)
 			(thermal_bridge_width 0.5)
@@
 		(min_thickness 0.2)
 		(filled_areas_thickness no)
-		(fill
+		(fill yes
 			(thermal_gap 0.2)
 			(thermal_bridge_width 0.5)
@@
 		(min_thickness 0.2)
 		(filled_areas_thickness no)
-		(fill
+		(fill yes
 			(thermal_gap 0.2)
 			(thermal_bridge_width 0.5)
@@
 		(min_thickness 0.2)
 		(filled_areas_thickness no)
-		(fill
+		(fill yes
 			(thermal_gap 0.2)
 			(thermal_bridge_width 0.5)
@@
 		(min_thickness 0.2)
 		(filled_areas_thickness no)
-		(fill
+		(fill yes
 			(thermal_gap 0.2)
 			(thermal_bridge_width 0.5)

Commit message: weW
Parts:
- added C28: 10n, hellen-one-common:C0603, F.Cu at (173.2, 63.5)
- added C29: 100n, hellen-one-common:C0603, F.Cu at (175.5, 56.0)
- added C30: 10n, hellen-one-common:C0603, F.Cu at (175.3, 62.5)
- added C31: 100n, hellen-one-common:C0603, F.Cu at (176.5, 52.0)
- added C32: 1u, hellen-one-common:C0603, F.Cu at (178.0, 52.0)
- added F10: 50mA, Fuse:Fuse_0603_1608Metric, B.Cu at (168.0, 57.0)
- added U11: VNLD5160TR-E, Package_SO:SOIC-8_3.9x4.9mm_P1.27mm, F.Cu at (187.5, 23.0)
- added U9: VNLD5160TR-E, Package_SO:SOIC-8_3.9x4.9mm_P1.27mm, F.Cu at (127.0, 51.5)
- D1, D2, D3, D4, F5, F6, F7, F8, F9, R13, R14, R16, R17, R18, R19, R2, R20, R21, R22, R23, R24, R25, R26, R27, R28, R29, R3, R30, R31, R32, R33, R34, R35, R36, R37, R38, R39, R40, R41, R42, R43, R44, R45, R46, R47, R48, R49, R50, R51, R52, R53: moved to B.Cu
- moved J21 104.7 mm to (176.0, 7.35), turned to 180 degrees
- moved D5 98.3 mm to (55.0, 72.2), turned to -90 degrees
- moved Q7 96.4 mm to (64.0, 65.7), turned to -90 degrees
- moved R52 96.3 mm to (190.0, 17.0), turned to -90 degrees
- moved R53 95.1 mm to (187.0, 17.0), turned to -90 degrees
- moved R54 89.5 mm to (61.0, 65.7), turned to 90 degrees
- moved R15 85.8 mm to (64.0, 61.7), turned to 180 degrees
- moved R13 78.2 mm to (159.5, 49.5), turned to -90 degrees
- moved M1 77.5 mm to (177.5, 20.9), turned to 180 degrees
- moved U10 76.5 mm to (63.0, 75.0), turned to -90 degrees
- moved R14 75.9 mm to (156.5, 49.5), turned to -90 degrees
- moved J22 74.4 mm to (159.5, 9.35), turned to -90 degrees
- moved L1 74.2 mm to (175.0, 67.0), turned to 90 degrees
- moved L2 72.6 mm to (173.0, 67.0), turned to 90 degrees
- moved R2 72.5 mm to (175.5, 67.0), turned to 180 degrees
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
Commit message: weW
Parts:
- renumbered F5 to F4, F6 to F5, F7 to F6, F8 to F7, F9 to F8, F10 to F9
Connections:
- R13 pad 2: Net-(U1-IN1) -> (no net)
- R14 pad 2: Net-(U1-IN2) -> (no net)
- R18 pad 2: Net-(U2-IN1) -> (no net)
- R19 pad 2: Net-(U2-IN2) -> (no net)
Changed lines of the file:
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@@
 			(layers "B.Cu" "B.Paste" "B.Mask")
 			(roundrect_rratio 0.1)
-			(net 217 "Net-(U2-IN1)")
 			(pintype "passive")
 		)
@@
 		(descr "Fuse SMD 0603 (1608 Metric), square (rectangular) end terminal, IPC_7351 nominal, (Body size source: http://www.tortai-tech.com/upload/download/2011102023233369053.pdf), generated with kicad-footprint-generator")
 		(tags "fuse")
-		(property "Reference" "F10"
+		(property "Reference" "F9"
 			(at -3 0 0)
 			(layer "B.SilkS")
@@
 			(layers "B.Cu" "B.Paste" "B.Mask")
 			(roundrect_rratio 0.1)
-			(net 218 "Net-(U2-IN2)")
 			(pintype "passive")
 		)
@@
 		(descr "Fuse SMD 0603 (1608 Metric), square (rectangular) end terminal, IPC_7351 nominal, (Body size source: http://www.tortai-tech.com/upload/download/2011102023233369053.pdf), generated with kicad-footprint-generator")
 		(tags "fuse")
-		(property "Reference" "F8"
+		(property "Reference" "F7"
 			(at -2.5 0 0)
 			(layer "B.SilkS")
@@
 			(layers "B.Cu" "B.Paste" "B.Mask")
 			(roundrect_rratio 0.1)
-			(net 216 "Net-(U1-IN2)")
 			(pintype "passive")
 		)
@@
 		(descr "Fuse SMD 0603 (1608 Metric), square (rectangular) end terminal, IPC_7351 nominal, (Body size source: http://www.tortai-tech.com/upload/download/2011102023233369053.pdf), generated with kicad-footprint-generator")
 		(tags "fuse")
-		(property "Reference" "F6"
+		(property "Reference" "F5"
 			(at -2.5 0 0)
 			(layer "B.SilkS")
@@
 		(descr "Fuse SMD 0603 (1608 Metric), square (rectangular) end terminal, IPC_7351 nominal, (Body size source: http://www.tortai-tech.com/upload/download/2011102023233369053.pdf), generated with kicad-footprint-generator")
 		(tags "fuse")
-		(property "Reference" "F5"
+		(property "Reference" "F4"
 			(at -2.5 0 0)
 			(layer "B.SilkS")
@@
 		(descr "Fuse SMD 0603 (1608 Metric), square (rectangular) end terminal, IPC_7351 nominal, (Body size source: http://www.tortai-tech.com/upload/download/2011102023233369053.pdf), generated with kicad-footprint-generator")
 		(tags "fuse")
-		(property "Reference" "F9"
+		(property "Reference" "F8"
 			(at -2.5 0 0)
 			(layer "B.SilkS")
@@
 			(layers "B.Cu" "B.Paste" "B.Mask")
 			(roundrect_rratio 0.1)
-			(net 215 "Net-(U1-IN1)")
 			(pintype "passive")
 		)
@@
 		(descr "Fuse SMD 0603 (1608 Metric), square (rectangular) end terminal, IPC_7351 nominal, (Body size source: http://www.tortai-tech.com/upload/download/2011102023233369053.pdf), generated with kicad-footprint-generator")
 		(tags "fuse")
-		(property "Reference" "F7"
+		(property "Reference" "F6"
 			(at -2.5 0 0)
 			(layer "B.SilkS")

Commit message: weW
Parts:
- removed C1, C3: 10n, hellen-one-common:C0603
- removed C2, C4: 100n, hellen-one-common:C0603
- removed C5: 1u, hellen-one-common:C0603
- removed F4: 50mA, Fuse:Fuse_0603_1608Metric
- removed U1, U2: VNLD5160TR-E, Package_SO:SOIC-8_3.9x4.9mm_P1.27mm
- R17, R18, R19: value 4.7k -> 22
- R20, R21: value 4.7k -> 0; footprint hellen-one-common:R0603 -> Resistor_SMD:R_2512_6332Metric
- R22, R28: value 22 -> 0; footprint hellen-one-common:R0603 -> Resistor_SMD:R_2512_6332Metric
- R25: value 0 -> 22; footprint Resistor_SMD:R_2512_6332Metric -> hellen-one-common:R0603
- R29, R30: value 22 -> 4.7k
- R31, R32, R33: value 0 -> 4.7k; footprint Resistor_SMD:R_2512_6332Metric -> hellen-one-common:R0603
- renumbered F9 to F10, F4 to F5, F5 to F6, F6 to F7, F7 to F8, F8 to F9
Connections:
- F5 pad 2: /IGN2 -> /IGN1
- F6 pad 2: /IGN3 -> /IGN2
- F7 pad 2: /IGN4 -> /IGN3
- F8 pad 2: /IGN5 -> /IGN4
- F9 pad 2: /IGN6 -> /IGN5
- R13 pad 1: /LS1 -> /LS_HOT2
- R13 pad 2: (no net) -> Net-(U7-IN1)
- R14 pad 1: /LS2 -> /LS_HOT1
- R14 pad 2: (no net) -> Net-(U7-IN2)
- R17 pad 1: /LS2 -> Net-(Q1-G)
- R17 pad 2: PIN114 -> Net-(F5-Pad1)
- R18 pad 1: /LS3 -> Net-(Q2-G)
- R18 pad 2: (no net) -> Net-(F6-Pad1)
- R19 pad 1: /LS4 -> Net-(Q3-G)
- R19 pad 2: (no net) -> Net-(F7-Pad1)
- R20 pad 1: /LS3 -> Net-(F5-Pad1)
- R20 pad 2: PIN114 -> PIN13
- R21 pad 1: /LS4 -> Net-(F6-Pad1)
- R21 pad 2: PIN114 -> PIN12
- R22 pad 1: Net-(Q1-G) -> Net-(F7-Pad1)
- R22 pad 2: Net-(F4-Pad1) -> PIN10
- R23 pad 1: Net-(Q2-G) -> Net-(Q4-G)
- R23 pad 2: Net-(F5-Pad1) -> Net-(F8-Pad1)
- R24 pad 1: Net-(Q3-G) -> Net-(Q5-G)
- R24 pad 2: Net-(F6-Pad1) -> Net-(F9-Pad1)
- R25 pad 1: Net-(F4-Pad1) -> Net-(Q6-G)
- R25 pad 2: PIN13 -> (no net)
- R26 pad 1: Net-(F5-Pad1) -> Net-(F8-Pad1)
- R26 pad 2: PIN12 -> PIN9
- R27 pad 1: Net-(F6-Pad1) -> Net-(F9-Pad1)
- R27 pad 2: PIN10 -> PIN11
- R28 pad 1: Net-(Q4-G) -> (no net)
- R28 pad 2: Net-(F7-Pad1) -> PIN8
- R29 pad 1: Net-(Q5-G) -> /INJ1
- R29 pad 2: Net-(F8-Pad1) -> PIN114
- R30 pad 1: Net-(Q6-G) -> /INJ3
- R30 pad 2: Net-(F9-Pad1) -> PIN114
- R31 pad 1: Net-(F7-Pad1) -> /INJ5
- R31 pad 2: PIN9 -> PIN114
- R32 pad 1: Net-(F8-Pad1) -> /INJ2
- R32 pad 2: PIN11 -> PIN114
- R33 pad 1: Net-(F9-Pad1) -> /INJ4
- R33 pad 2: PIN8 -> PIN114
- R34 pad 1: E6INJ7CANRX -> /INJ6
- R34 pad 2: Net-(U3-IN1) -> PIN114
- R35 pad 1: E7INJ8CANTX -> /LS_HOT1
- R36 pad 1: E7INJ8CANTX -> /LS_HOT2
- R36 pad 2: Net-(U3-IN2) -> PIN114
- R37 pad 1: E6INJ7CANRX -> /LS3
- R38 pad 1: /INJ1 -> /LS2
- R38 pad 2: Net-(U6-IN1) -> PIN114
- R39 pad 1: /INJ1 -> /LS4
- R40 pad 1: /INJ2 -> E6INJ7CANRX
- R41 pad 1: /INJ2 -> E7INJ8CANTX
- R41 pad 2: Net-(U6-IN2) -> PIN114
- R42 pad 1: /INJ3 -> /LS3
- R42 pad 2: Net-(U4-IN1) -> (no net)
- R43 pad 1: /INJ3 -> /LS4
- R43 pad 2: PIN114 -> (no net)
- R44 pad 1: /INJ4 -> /LS1
- R44 pad 2: PIN114 -> Net-(U3-IN1)
- R45 pad 1: /INJ4 -> /LS2
- R45 pad 2: Net-(U4-IN2) -> Net-(U3-IN2)
- R46 pad 1: /INJ5 -> /INJ1
- R46 pad 2: Net-(U5-IN1) -> Net-(U4-IN1)
- R47 pad 1: /INJ5 -> /INJ2
- R47 pad 2: PIN114 -> Net-(U4-IN2)
- R48 pad 1: /INJ6 -> /INJ3
- R48 pad 2: Net-(U5-IN2) -> Net-(U5-IN1)
- R49 pad 1: /INJ6 -> /INJ4
- R49 pad 2: PIN114 -> Net-(U5-IN2)
- R50 pad 1: /LS_HOT2 -> /INJ5
- R50 pad 2: Net-(U7-IN1) -> Net-(U6-IN1)
- R51 pad 1: /LS_HOT2 -> /INJ6
- R51 pad 2: PIN114 -> Net-(U6-IN2)
- R52 pad 1: /LS_HOT1 -> E6INJ7CANRX
- R52 pad 2: Net-(U7-IN2) -> (no net)
- R53 pad 1: /LS_HOT1 -> E7INJ8CANTX
- R53 pad 2: PIN114 -> (no net)
- U3 pad 6: PIN51 -> PIN15
- U3 pad 8: PIN50 -> PIN14
- U4 pad 6: PIN47 -> PIN45
- U4 pad 8: PIN46 -> PIN44
- U5 pad 6: PIN49 -> PIN47
- U5 pad 8: PIN48 -> PIN46
- U6 pad 6: PIN45 -> PIN49
- U6 pad 8: PIN44 -> PIN48

Commit message: weW
Parts:
- renumbered C28 to C1, C30 to C2, C29 to C3
Changed lines of the file:
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@@
 		(layer "F.Cu")
 		(at 173.209999 63.5 180)
-		(property "Reference" "C28"
+		(property "Reference" "C1"
 			(at -1.290001 -0.74013 180)
 			(unlocked yes)
@@
 		(layer "F.Cu")
 		(at 175.290001 62.5)
-		(property "Reference" "C30"
+		(property "Reference" "C2"
 			(at 1.709999 1 180)
 			(unlocked yes)
@@
 		(layer "F.Cu")
 		(at 175.5 56)
-		(property "Reference" "C29"
+		(property "Reference" "C3"
 			(at -0.708119 -0.74013 0)
 			(unlocked yes)

Commit message: weW
Parts:
- renumbered C31 to C4, C32 to C5
Changed lines of the file:
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@@
 		(layer "F.Cu")
 		(at 178 52 -90)
-		(property "Reference" "C32"
+		(property "Reference" "C5"
 			(at -4 0.5 -90)
 			(unlocked yes)
@@
 		(layer "F.Cu")
 		(at 176.5 52 -90)
-		(property "Reference" "C31"
-			(at -4 0.5 -90)
+		(property "Reference" "C4"
+			(at -4 0.5 270)
 			(unlocked yes)
 			(layer "F.SilkS")
