File: greenenergyecu.kicad_pcb (KiCad board)
At the start: 4 copper layers, 164 x 118 mm, 103 parts, among them J21 Conn_01x05_Male, J22 USB_B_Mini, M1 Module-power_12and5V-0.3, M2 Module-knock-0.2, M3 Module-vr-discrete-0.5, M4 Module-vr-max9924-0.1, M5 Module-wbo-0.5, M6 Module:mega-mcu100/0.3, M7 Module-can-0.1, M8 Module-motor-driver-0.1, P1 368255-2, Q1 ISL9V3040D3ST, Q2 ISL9V3040D3ST, Q3 ISL9V3040D3ST, Q4 ISL9V3040D3ST, Q5 ISL9V3040D3ST, Q6 ISL9V3040D3ST, Q7 AO3400A, U10 BTS6143D, U11 VNLD5160TR-E, U3 VNLD5160TR-E, U4 VNLD5160TR-E, U5 VNLD5160TR-E, U6 VNLD5160TR-E, U7 VNLD5160TR-E, U8 MAX31855KASA, U9 VNLD5160TR-E

Commit message: weW
Parts:
- renumbered F5 to F844, F6 to F845, F7 to F846, F8 to F847, F9 to F848, F10 to F849, Q1 to Q841, Q2 to Q842, Q3 to Q843, Q4 to Q844, Q5 to Q845, Q6 to Q846, R17 to R867, R18 to R868, R19 to R869, R20 to R870, R21 to R871, R22 to R872, R23 to R873, R24 to R874, R25 to R875, R26 to R876, R27 to R877, R28 to R878, U11 to U2, U3 to U842, U9 to U843, U7 to U844, U8 to U846, U4 to U847, U5 to U848, U6 to U849
Changed lines of the file:
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@@
 		(descr "SOIC, 8 Pin (JEDEC MS-012AA, https://www.analog.com/media/en/package-pcb-resources/package/pkg_pdf/soic_narrow-r/r_8.pdf), generated with kicad-footprint-generator ipc_gullwing_generator.py")
 		(tags "SOIC SO")
-		(property "Reference" "U8"
+		(property "Reference" "U846"
 			(at 0 -3.5 90)
 			(layer "F.SilkS")
@@
 		(descr "TO-252/DPAK SMD package, http://www.infineon.com/cms/en/product/packages/PG-TO252/PG-TO252-3-1/")
 		(tags "DPAK TO-252 DPAK-3 TO-252-3 SOT-428")
-		(property "Reference" "Q1"
-			(at 0 -4.5 90)
+		(property "Reference" "Q841"
+			(at -4.565 0.22 90)
 			(layer "F.SilkS")
 			(effects
@@
 		(descr "SOIC, 8 Pin (JEDEC MS-012AA, https://www.analog.com/media/en/package-pcb-resources/package/pkg_pdf/soic_narrow-r/r_8.pdf), generated with kicad-footprint-generator ipc_gullwing_generator.py")
 		(tags "SOIC SO")
-		(property "Reference" "U3"
-			(at 0 -3.4 90)
+		(property "Reference" "U842"
+			(at -5 0 180)
 			(layer "F.SilkS")
 			(effects
@@
 		(descr "SOIC, 8 Pin (JEDEC MS-012AA, https://www.analog.com/media/en/package-pcb-resources/package/pkg_pdf/soic_narrow-r/r_8.pdf), generated with kicad-footprint-generator ipc_gullwing_generator.py")
 		(tags "SOIC SO")
-		(property "Reference" "U5"
-			(at 0 -3.4 90)
+		(property "Reference" "U848"
+			(at -5 0 180)
 			(layer "F.SilkS")
 			(effects
@@
 		(descr "TO-252/DPAK SMD package, http://www.infineon.com/cms/en/product/packages/PG-TO252/PG-TO252-3-1/")
 		(tags "DPAK TO-252 DPAK-3 TO-252-3 SOT-428")
-		(property "Reference" "Q5"
-			(at 0 -4.5 90)
+		(property "Reference" "Q845"
+			(at -4.565 0 90)
 			(layer "F.SilkS")
 			(effects
@@
 		(descr "TO-252/DPAK SMD package, http://www.infineon.com/cms/en/product/packages/PG-TO252/PG-TO252-3-1/")
 		(tags "DPAK TO-252 DPAK-3 TO-252-3 SOT-428")
-		(property "Reference" "Q2"
-			(at 0 -4.5 90)
+		(property "Reference" "Q842"
+			(at -4.565 -0.085 90)
 			(layer "F.SilkS")
 			(effects
@@
 		(descr "SOIC, 8 Pin (JEDEC MS-012AA, https://www.analog.com/media/en/package-pcb-resources/package/pkg_pdf/soic_narrow-r/r_8.pdf), generated with kicad-footprint-generator ipc_gullwing_generator.py")
 		(tags "SOIC SO")
-		(property "Reference" "U7"
-			(at 0 -3.4 90)
+		(property "Reference" "U844"
+			(at -5 0.405 180)
 			(layer "F.SilkS")
 			(effects
@@
 		(descr "SOIC, 8 Pin (JEDEC MS-012AA, https://www.analog.com/media/en/package-pcb-resources/package/pkg_pdf/soic_narrow-r/r_8.pdf), generated with kicad-footprint-generator ipc_gullwing_generator.py")
 		(tags "SOIC SO")
-		(property "Reference" "U4"
-			(at 0 -3.4 90)
+		(property "Reference" "U847"
+			(at -5 0 180)
 			(layer "F.SilkS")
 			(effects
@@
 		(descr "TO-252/DPAK SMD package, http://www.infineon.com/cms/en/product/packages/PG-TO252/PG-TO252-3-1/")
 		(tags "DPAK TO-252 DPAK-3 TO-252-3 SOT-428")
-		(property "Reference" "Q3"
-			(at 0 -4.5 90)
+		(property "Reference" "Q843"
+			(at -4.065 -0.39 90)
 			(layer "F.SilkS")
 			(effects
@@
 		(descr "TO-252/DPAK SMD package, http://www.infineon.com/cms/en/product/packages/PG-TO252/PG-TO252-3-1/")
 		(tags "DPAK TO-252 DPAK-3 TO-252-3 SOT-428")
-		(property "Reference" "Q6"
-			(at 5.935 -0.305 90)
+		(property "Reference" "Q846"
+			(at -4.565 0.195 90)
 			(layer "F.SilkS")
 			(effects
@@
 		(descr "SOIC, 8 Pin (JEDEC MS-012AA, https://www.analog.com/media/en/package-pcb-resources/package/pkg_pdf/soic_narrow-r/r_8.pdf), generated with kicad-footprint-generator ipc_gullwing_generator.py")
 		(tags "SOIC SO")
-		(property "Reference" "U11"
+		(property "Reference" "U2"
 			(at 0 -3.4 90)
 			(layer "F.SilkS")
@@
 		(descr "SOIC, 8 Pin (JEDEC MS-012AA, https://www.analog.com/media/en/package-pcb-resources/package/pkg_pdf/soic_narrow-r/r_8.pdf), generated with kicad-footprint-generator ipc_gullwing_generator.py")
 		(tags "SOIC SO")
-		(property "Reference" "U9"
-			(at 0 -3.4 90)
+		(property "Reference" "U843"
+			(at -5 0 180)
 			(layer "F.SilkS")
 			(effects
@@
 		(descr "TO-252/DPAK SMD package, http://www.infineon.com/cms/en/product/packages/PG-TO252/PG-TO252-3-1/")
 		(tags "DPAK TO-252 DPAK-3 TO-252-3 SOT-428")
-		(property "Reference" "Q4"
-			(at 0 -4.5 90)
+		(property "Reference" "Q844"
+			(at -4.565 -0.195 90)
 			(layer "F.SilkS")
 			(effects
@@
 		(descr "SOIC, 8 Pin (JEDEC MS-012AA, https://www.analog.com/media/en/package-pcb-resources/package/pkg_pdf/soic_narrow-r/r_8.pdf), generated with kicad-footprint-generator ipc_gullwing_generator.py")
 		(tags "SOIC SO")
-		(property "Reference" "U6"
-			(at 0 -3.4 90)
+		(property "Reference" "U849"
+			(at -5 -0.635 180)
 			(layer "F.SilkS")
 			(effects
@@
 		(descr "Resistor SMD 2512 (6332 Metric), square (rectangular) end terminal, IPC_7351 nominal, (Body size source: IPC-SM-782 page 72, https://www.pcb-3d.com/wordpress/wp-content/uploads/ipc-sm-782a_amendment_1_and_2.pdf), generated with kicad-footprint-generator")
 		(tags "resistor")
-		(property "Reference" "R28"
+		(property "Reference" "R878"
 			(at 0 2.62 90)
 			(layer "B.SilkS")
@@
 		(layer "B.Cu")
 		(at 135.5 59 180)
-		(property "Reference" "R18"
+		(property "Reference" "R868"
 			(at 4 0.5 180)
 			(unlocked yes)
@@
 		(descr "Fuse SMD 0603 (1608 Metric), square (rectangular) end terminal, IPC_7351 nominal, (Body size source: http://www.tortai-tech.com/upload/download/2011102023233369053.pdf), generated with kicad-footprint-generator")
 		(tags "fuse")
-		(property "Reference" "F10"
+		(property "Reference" "F849"
 			(at -3 0 0)
 			(layer "B.SilkS")
@@
 		(layer "B.Cu")
 		(at 143.5 59 180)
-		(property "Reference" "R19"
+		(property "Reference" "R869"
 			(at 4 0.5 180)
 			(unlocked yes)
@@
 		(layer "B.Cu")
 		(at 127 59 180)
-		(property "Reference" "R17"
+		(property "Reference" "R867"
 			(at 4 0.5 180)
 			(unlocked yes)
@@
 		(layer "B.Cu")
 		(at 152 59 180)
-		(property "Reference" "R23"
+		(property "Reference" "R873"
 			(at 4 0.5 180)
 			(unlocked yes)
@@
 		(descr "Resistor SMD 2512 (6332 Metric), square (rectangular) end terminal, IPC_7351 nominal, (Body size source: IPC-SM-782 page 72, https://www.pcb-3d.com/wordpress/wp-content/uploads/ipc-sm-782a_amendment_1_and_2.pdf), generated with kicad-footprint-generator")
 		(tags "resistor")
-		(property "Reference" "R20"
+		(property "Reference" "R870"
 			(at 0.0375 4 90)
 			(layer "B.SilkS")
@@
 		(descr "Fuse SMD 0603 (1608 Metric), square (rectangular) end terminal, IPC_7351 nominal, (Body size source: http://www.tortai-tech.com/upload/download/2011102023233369053.pdf), generated with kicad-footprint-generator")
 		(tags "fuse")
-		(property "Reference" "F8"
+		(property "Reference" "F847"
 			(at -2.5 0 0)
 			(layer "B.SilkS")
@@
 		(descr "Resistor SMD 2512 (6332 Metric), square (rectangular) end terminal, IPC_7351 nominal, (Body size source: IPC-SM-782 page 72, https://www.pcb-3d.com/wordpress/wp-content/uploads/ipc-sm-782a_amendment_1_and_2.pdf), generated with kicad-footprint-generator")
 		(tags "resistor")
-		(property "Reference" "R26"
+		(property "Reference" "R876"
 			(at 0 3 90)
 			(layer "B.SilkS")
@@
 		(descr "Fuse SMD 0603 (1608 Metric), square (rectangular) end terminal, IPC_7351 nominal, (Body size source: http://www.tortai-tech.com/upload/download/2011102023233369053.pdf), generated with kicad-footprint-generator")
 		(tags "fuse")
-		(property "Reference" "F6"
+		(property "Reference" "F845"
 			(at -2.5 0 0)
 			(layer "B.SilkS")
@@
 		(descr "Fuse SMD 0603 (1608 Metric), square (rectangular) end terminal, IPC_7351 nominal, (Body size source: http://www.tortai-tech.com/upload/download/2011102023233369053.pdf), generated with kicad-footprint-generator")
 		(tags "fuse")
-		(property "Reference" "F5"
+		(property "Reference" "F844"
 			(at -2.5 0 0)
 			(layer "B.SilkS")
@@
 		(descr "Fuse SMD 0603 (1608 Metric), square (rectangular) end terminal, IPC_7351 nominal, (Body size source: http://www.tortai-tech.com/upload/download/2011102023233369053.pdf), generated with kicad-footprint-generator")
 		(tags "fuse")
-		(property "Reference" "F9"
+		(property "Reference" "F848"
 			(at -2.5 0 0)
 			(layer "B.SilkS")
@@
 		(layer "B.Cu")
 		(at 160 59 180)
-		(property "Reference" "R24"
+		(property "Reference" "R874"
 			(at 3.5 0.5 180)
 			(unlocked yes)
@@
 		(descr "Fuse SMD 0603 (1608 Metric), square (rectangular) end terminal, IPC_7351 nominal, (Body size source: http://www.tortai-tech.com/upload/download/2011102023233369053.pdf), generated with kicad-footprint-generator")
 		(tags "fuse")
-		(property "Reference" "F7"
+		(property "Reference" "F846"
 			(at -2.5 0 0)
 			(layer "B.SilkS")
@@
 		(descr "Resistor SMD 2512 (6332 Metric), square (rectangular) end terminal, IPC_7351 nominal, (Body size source: IPC-SM-782 page 72, https://www.pcb-3d.com/wordpress/wp-content/uploads/ipc-sm-782a_amendment_1_and_2.pdf), generated with kicad-footprint-generator")
 		(tags "resistor")
-		(property "Reference" "R22"
+		(property "Reference" "R872"
 			(at 0 2.62 90)
 			(layer "B.SilkS")
@@
 		(descr "Resistor SMD 2512 (6332 Metric), square (rectangular) end terminal, IPC_7351 nominal, (Body size source: IPC-SM-782 page 72, https://www.pcb-3d.com/wordpress/wp-content/uploads/ipc-sm-782a_amendment_1_and_2.pdf), generated with kicad-footprint-generator")
 		(tags "resistor")
-		(property "Reference" "R27"
+		(property "Reference" "R877"
 			(at 0 3 90)
 			(layer "B.SilkS")
@@
 		(descr "Resistor SMD 2512 (6332 Metric), square (rectangular) end terminal, IPC_7351 nominal, (Body size source: IPC-SM-782 page 72, https://www.pcb-3d.com/wordpress/wp-content/uploads/ipc-sm-782a_amendment_1_and_2.pdf), generated with kicad-footprint-generator")
 		(tags "resistor")
-		(property "Reference" "R21"
+		(property "Reference" "R871"
 			(at 0 3 90)
 			(layer "B.SilkS")
@@
 		(layer "B.Cu")
 		(at 168 59 180)
-		(property "Reference" "R25"
+		(property "Reference" "R875"
 			(at 4 0.5 180)
 			(unlocked yes)
