File: greenenergyecu.kicad_pcb (KiCad board)
At the start: 4 copper layers, 164 x 118 mm, 129 parts, among them J22 USB_B_Mini, M1 Module-power_12and5V-0.3, M2 Module-knock-0.2, M3 Module-vr-discrete-0.5, M4 Module-vr-max9924-0.1, M5 Module-wbo-0.5, M6 Module:mega-mcu100/0.3, M7 Module-can-0.1, M8 Module-motor-driver-0.1, M9 Module-ign8-0.2, P1 368255-2, Q1 AO3400A, Q3 ISL9V3040D3ST, Q841 ISL9V3040D3ST, Q842 ISL9V3040D3ST, Q843 ISL9V3040D3ST, Q844 ISL9V3040D3ST, Q845 ISL9V3040D3ST, Q846 ISL9V3040D3ST, Q847 ISL9V3040D3ST, Q849 ISL9V3040D3ST, Q900 ISL9V3040D3ST, Q901 ISL9V3040D3ST, Q902 ISL9V3040D3ST, Q903 ISL9V3040D3ST, Q904 ISL9V3040D3ST, Q905 ISL9V3040D3ST, Q906 ISL9V3040D3ST, Q907 ISL9V3040D3ST, U1 BTS6143D, U842 VNLD5160TR-E, U843 VNLD5160TR-E, U846 MAX31855KASA

Commit message: tilo
Connections:
- R1 pad 2: /LSH/IN2 -> /DC2_DIR
Routing:
- net +12V: track 173.5 -> 322.0 mm
- net /DC2_DIR: track 95.7 -> 96.3 mm
- net GND: vias 104 -> 112
- added copper zone on F.Cu, net GND

Commit message: tilo
Routing:
- added copper zone on In2.Cu, net GND
- removed copper zone on In2.Cu, net +12V
Changed lines of the file:
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@@
 		(min_thickness 0.254)
 		(filled_areas_thickness no)
-		(fill
+		(fill yes
 			(thermal_gap 0.508)
 			(thermal_bridge_width 0.508)
@@
 		(min_thickness 0.2)
 		(filled_areas_thickness no)
-		(fill
+		(fill yes
 			(thermal_gap 0.2)
 			(thermal_bridge_width 0.5)
@@
 	)
 	(zone
-		(net 125)
-		(net_name "+12V")
+		(net 95)
+		(net_name "GND")
 		(layer "In2.Cu")
-		(hatch edge 0.5)
+		(hatch edge 0.508)
 		(priority 3)
-		(connect_pads
-			(clearance 0)
-		)
-		(min_thickness 0.25)
-		(filled_areas_thickness no)
-		(fill
-			(thermal_gap 0.5)
-			(thermal_bridge_width 0.5)
-		)
-		(polygon
-			(pts
-				(xy 37.156 -20.628) (xy 220.219 -18.769) (xy 218.093 130.02) (xy 36.89 120.986)
+		(connect_pads yes
+			(clearance 0.2)
+		)
+		(min_thickness 0.254)
+		(filled_areas_thickness no)
+		(fill yes
+			(thermal_gap 0.508)
+			(thermal_bridge_width 0.508)
+		)
+		(polygon
+			(pts
+				(xy 34.29 -26.035) (xy 215.265 -25.4) (xy 214.63 126.365) (xy 36.195 123.825)
 			)
 		)
@@
 		(min_thickness 0.2)
 		(filled_areas_thickness no)
-		(fill
+		(fill yes
 			(thermal_gap 0.2)
 			(thermal_bridge_width 0.5)
@@
 		(min_thickness 0.2)
 		(filled_areas_thickness no)
-		(fill
+		(fill yes
 			(thermal_gap 0.2)
 			(thermal_bridge_width 0.5)
@@
 		(min_thickness 0.2)
 		(filled_areas_thickness no)
-		(fill
+		(fill yes
 			(thermal_gap 0.2)
 			(thermal_bridge_width 0.5)
@@
 		(min_thickness 0.2)
 		(filled_areas_thickness no)
-		(fill
+		(fill yes
 			(thermal_gap 0.2)
 			(thermal_bridge_width 0.5)
@@
 		(min_thickness 0.2)
 		(filled_areas_thickness no)
-		(fill
-			(thermal_gap 0.2)
-			(thermal_bridge_width 0.5)
+		(fill yes
+			(thermal_gap 0.2)
+			(thermal_bridge_width 0.5)

Commit message: tilo
Routing:
- net GND: vias 112 -> 126
Changed lines of the file:
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@@
 	)
 	(via
+		(at 49.29 91.41)
+		(size 0.6)
+		(drill 0.3)
+		(layers "F.Cu" "B.Cu")
+		(free yes)
+		(net 95)
+	)
+	(via
 		(at 86.97999 12.27999)
 		(size 0.15)
@@
 	)
 	(via
+		(at 47.94 15.2)
+		(size 0.6)
+		(drill 0.3)
+		(layers "F.Cu" "B.Cu")
+		(free yes)
+		(net 95)
+	)
+	(via
 		(at 190.67 29.658)
 		(size 0.8)
@@
 	)
 	(via
+		(at 48.78 55.07)
+		(size 0.6)
+		(drill 0.3)
+		(layers "F.Cu" "B.Cu")
+		(free yes)
+		(net 95)
+	)
+	(via
 		(at 166.437 74.51)
 		(size 0.8)
@@
 	)
 	(via
+		(at 189.42 -5.15)
+		(size 0.6)
+		(drill 0.3)
+		(layers "F.Cu" "B.Cu")
+		(free yes)
+		(net 95)
+	)
+	(via
 		(at 168.4 18.430002)
 		(size 0.15)
@@
 	)
 	(via
+		(at 92.44 -5.22)
+		(size 0.6)
+		(drill 0.3)
+		(layers "F.Cu" "B.Cu")
+		(free yes)
+		(net 95)
+	)
+	(via
 		(at 172.18275 74.10475)
 		(size 0.8)
@@
 	)
 	(via
+		(at 206.78 7.13)
+		(size 0.6)
+		(drill 0.3)
+		(layers "F.Cu" "B.Cu")
+		(free yes)
+		(net 95)
+	)
+	(via
 		(at 126.6495 67.6835)
 		(size 0.15)
@@
 	)
 	(via
+		(at 129.66 -4.98)
+		(size 0.6)
+		(drill 0.3)
+		(layers "F.Cu" "B.Cu")
+		(free yes)
+		(net 95)
+	)
+	(via
 		(at 133.882 10.554)
 		(size 0.3)
@@
 	)
 	(via
+		(at 207.16 92.67)
+		(size 0.6)
+		(drill 0.3)
+		(layers "F.Cu" "B.Cu")
+		(free yes)
+		(net 95)
+	)
+	(via
 		(at 141.80125 73.71375)
 		(size 0.8)
@@
 	)
 	(via
+		(at 48.43 40.43)
+		(size 0.6)
+		(drill 0.3)
+		(layers "F.Cu" "B.Cu")
+		(free yes)
+		(net 95)
+	)
+	(via
 		(at 86.97999 33.42999)
 		(size 0.15)
@@
 	)
 	(via
+		(at 61.9 -4.68)
+		(size 0.6)
+		(drill 0.3)
+		(layers "F.Cu" "B.Cu")
+		(free yes)
+		(net 95)
+	)
+	(via
 		(at 121.824 10.682)
 		(size 0.3)
@@
 	)
 	(via
+		(at 48.78 66.09)
+		(size 0.6)
+		(drill 0.3)
+		(layers "F.Cu" "B.Cu")
+		(free yes)
+		(net 95)
+	)
+	(via
 		(at 164.5975 73.9575)
 		(size 0.8)
@@
 	)
 	(via
+		(at 207.26 38.23)
+		(size 0.6)
+		(drill 0.3)
+		(layers "F.Cu" "B.Cu")
+		(free yes)
+		(net 95)
+	)
+	(via
+		(at 206.64 60.12)
+		(size 0.6)
+		(drill 0.3)
+		(layers "F.Cu" "B.Cu")
+		(free yes)
+		(net 95)
+	)
+	(via
 		(at 162.174 9.636)
 		(size 0.3)
@@
 	)
 	(via
+		(at 48.6 79.52)
+		(size 0.6)
+		(drill 0.3)
+		(layers "F.Cu" "B.Cu")
+		(free yes)
+		(net 95)
+	)
+	(via
 		(at 59.957999 80.638999)
 		(size 0.3)
@@
 			)
 		)
+	)
+	(zone
+		(net 0)
+		(net_name "")
+		(layer "B.Mask")
+		(hatch edge 0.508)
+		(priority 1)
+		(connect_pads
+			(clearance 0.2)
+		)
+		(min_thickness 0.2)
+		(filled_areas_thickness no)
+		(fill yes
+			(thermal_gap 0.2)
+			(thermal_bridge_width 0.5)
+		)
+		(polygon
+			(pts
+				(xy 51.628762 10.560203) (xy 52.503762 10.410203) (xy 53.428762 10.185203) (xy 54.253762 9.935203)
+				(xy 54.903762 9.685203) (xy 55.528762 9.410203) (xy 56.253762 9.060203) (xy 57.053762 8.610203)
+				(xy 57.878762 8.035203) (xy 58.628762 7.460203) (xy 59.253762 6.885203) (xy 59.953762 6.185203)
+				(xy 60.578762 5.435203) (xy 61.028762 4.810203) (xy 61.478762 4.135203) (xy 61.853762 3.485203)
+				(xy 62.228762 2.760203) (xy 62.578762 1.935203) (xy 62.953762 0.935203) (xy 63.203762 -0.039797)
+				(xy 63.353762 -0.889797) (xy 63.453762 -1.639797) (xy 63.478762 -1.864797) (xy 58.003762 -1.864797)
+				(xy 57.378762 -0.839797) (xy 55.628762 2.160203) (xy 51.603762 4.535203)
+			)
+		)
+	)
+	(zone
+		(net 0)
+		(net_name "")
+		(layer "B.Mask")
+		(hatch full 0.508)
+		(priority 1)
+		(connect_pads
+			(clearance 0.2)
+		)
+		(min_thickness 0.2)
+		(filled_areas_thickness no)
+		(fill yes
+			(thermal_gap 0.2)
+			(thermal_bridge_width 0.5)
+			(smoothing fillet)
+		)
+		(polygon
+			(pts
+				(xy 131.696583 -1.744997) (xy 197.171583 -1.744997) (xy 197.146583 -7.594997) (xy 58.496583 -7.569997)
+				(xy 58.496583 -1.744997)
+			)
+		)
+	)
+	(zone
+		(net 0)
+		(net_name "")
+		(layer "B.Mask")
+		(hatch full 0.508)
+		(priority 1)
+		(connect_pads
+			(clearance 0.2)
+		)
+		(min_thickness 0.2)
+		(filled_areas_thickness no)
+		(fill yes
+			(thermal_gap 0.2)
+			(thermal_bridge_width 0.5)
+			(smoothing fillet)
+		)
+		(polygon
+			(pts
+				(xy 203.696583 96.405003) (xy 203.696583 97.580003) (xy 209.480418 97.586389) (xy 209.471583 5.055003)
+				(xy 203.671583 5.055003)
+			)
+		)
+	)
+	(zone
+		(net 0)
+		(net_name "")
+		(layer "B.Mask")
+		(hatch full 0.508)
+		(priority 1)
+		(connect_pads
+			(clearance 0.2)
+		)
+		(min_thickness 0.2)
+		(filled_areas_thickness no)
+		(fill yes
+			(thermal_gap 0.2)
+			(thermal_bridge_width 0.5)
+			(smoothing fillet)
+		)
+		(polygon
+			(pts
+				(xy 45.871583 96.055003) (xy 47.197002 97.455) (xy 51.672002 97.43) (xy 51.671583 4.905003) (xy 45.871583 4.905003)
+			)
+		)
+	)
+	(zone
+		(net 0)
+		(net_name "")
+		(layer "B.Mask")
+		(hatch edge 0.508)
+		(priority 1)
+		(connect_pads
+			(clearance 0.2)
+		)
+		(min_thickness 0.2)
+		(filled_areas_thickness no)
+		(fill yes
+			(thermal_gap 0.2)
+			(thermal_bridge_width 0.5)
+		)
+		(polygon
+			(pts
+				(xy 191.471583 -1.844997) (xy 191.621583 -0.969997) (xy 191.846583 -0.044997) (xy 192.096583 0.780003)
+				(xy 192.346583 1.430003) (xy 192.621583 2.055003) (xy 192.971583 2.780003) (xy 193.421583 3.580003)
+				(xy 193.996583 4.405003) (xy 194.571583 5.155003) (xy 195.146583 5.780003) (xy 195.846583 6.480003)
+				(xy 196.596583 7.105003) (xy 197.221583 7.555003) (xy 197.896583 8.005003) (xy 198.546583 8.380003)
+				(xy 199.271583 8.755003) (xy 200.096583 9.105003) (xy 201.096583 9.480003) (xy 202.071583 9.730003)
+				(xy 202.921583 9.880003) (xy 203.671583 9.980003) (xy 203.896583 10.005003) (xy 203.896583 4.530003)
+				(xy 202.871583 3.905003) (xy 199.871583 2.155003) (xy 197.496583 -1.869997)
+			)
+		)

Commit message: tilo
Connections:
- R325 pad 1: /INJ7 -> /INJ8
- R327 pad 1: /INJ8 -> /INJ7
Changed lines of the file:
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@@
 		(at 136.23001 55.03 180)
 		(property "Reference" "F843"
-			(at -4 0 90)
+			(at -0.11999 2.46 90)
 			(layer "F.SilkS")
 			(effects
@@
 		)
 		(fp_text user "${REFERENCE}"
-			(at -4 0 90)
+			(at -0.11999 2.46 90)
 			(layer "B.SilkS")
 			(effects
@@
 		(tags "DPAK TO-252 DPAK-3 TO-252-3 SOT-428")
 		(property "Reference" "Q841"
-			(at -4.565 0.22 90)
+			(at -4.98 -8.66 90)
 			(layer "F.SilkS")
 			(effects
@@
 		(at 140.79101 68.561 180)
 		(property "Reference" "F841"
-			(at -4 0 90)
+			(at -4.33899 -0.049 90)
 			(layer "F.SilkS")
 			(effects
@@
 		)
 		(fp_text user "${REFERENCE}"
-			(at -4 0 90)
+			(at -4.24899 -0.129 90)
 			(layer "B.SilkS")
 			(effects
@@
 		(at 79.671 67.574)
 		(property "Reference" "R843"
-			(at -1.235559 -0.653823 0)
+			(at 1.419 0.436 0)
 			(unlocked yes)
 			(layer "F.SilkS")
@@
 		(tags "DPAK TO-252 DPAK-3 TO-252-3 SOT-428")
 		(property "Reference" "Q845"
-			(at -4.565 0 90)
+			(at 1.12 -4.47 90)
 			(layer "F.SilkS")
 			(effects
@@
 		(tags "DPAK TO-252 DPAK-3 TO-252-3 SOT-428")
 		(property "Reference" "Q842"
-			(at -4.565 -0.085 90)
+			(at 0.665 -4.555 90)
 			(layer "F.SilkS")
 			(effects
@@
 		(tags "DPAK TO-252 DPAK-3 TO-252-3 SOT-428")
 		(property "Reference" "Q907"
-			(at 0 -4.5 90)
+			(at 0.23 -4.33 90)
 			(layer "F.SilkS")
 			(effects
@@
 		(tags "DPAK TO-252 DPAK-3 TO-252-3 SOT-428")
 		(property "Reference" "Q843"
-			(at -4.065 -0.39 90)
+			(at 0.0225 -4.6975 90)
 			(layer "F.SilkS")
 			(effects
@@
 		(tags "DPAK TO-252 DPAK-3 TO-252-3 SOT-428")
 		(property "Reference" "Q846"
-			(at -4.565 0.195 90)
+			(at -5.4175 -8.85 90)
 			(layer "F.SilkS")
 			(effects
@@
 		(at 112.836 43.585 180)
 		(property "Reference" "R842"
-			(at -2 2 180)
+			(at -1.584 -0.545 0)
 			(unlocked yes)
 			(layer "F.SilkS")
@@
 			(layers "F.Cu" "F.Paste" "F.Mask")
 			(roundrect_rratio 0.1)
-			(net 192 "/INJ8")
+			(net 193 "/INJ7")
 			(pintype "passive")
 		)
@@
 		(at 112.795 45.43)
 		(property "Reference" "R841"
-			(at -1 2 0)
+			(at 1.775 0.27 0)
 			(unlocked yes)
 			(layer "F.SilkS")
@@
 			(layers "F.Cu" "F.Paste" "F.Mask")
 			(roundrect_rratio 0.1)
-			(net 193 "/INJ7")
+			(net 192 "/INJ8")
 			(pintype "passive")
 		)
@@
 		(at 58.632 36.7205 90)
 		(property "Reference" "R3"
-			(at -1.235559 -0.653823 0)
+			(at -0.6195 -2.172 0)
 			(unlocked yes)
 			(layer "F.SilkS")
@@
 		(tags "DPAK TO-252 DPAK-3 TO-252-3 SOT-428")
 		(property "Reference" "Q849"
-			(at -5.43 -0.05 90)
+			(at 0.88 -4.33 90)
 			(layer "F.SilkS")
 			(effects
@@
 		(tags "DPAK TO-252 DPAK-3 TO-252-3 SOT-428")
 		(property "Reference" "Q847"
-			(at 0 -4.5 90)
+			(at -5.29 -8.1025 90)
 			(layer "F.SilkS")
 			(effects
@@
 		(at 61.092 33.880428 180)
 		(property "Reference" "R4"
-			(at -1.235559 -0.653823 180)
+			(at -0.988 1.990428 180)
 			(unlocked yes)
 			(layer "F.SilkS")
@@
 		(tags "DPAK TO-252 DPAK-3 TO-252-3 SOT-428")
 		(property "Reference" "Q844"
-			(at -4.565 -0.195 90)
+			(at -5.085 -8.615 90)
 			(layer "F.SilkS")
 			(effects
@@
 		(tags "resistor")
 		(property "Reference" "R878"
-			(at 0 2.62 90)
+			(at -0.34 -2.97 90)
 			(layer "B.SilkS")
 			(effects
@@
 		(at 196.65 31.38 180)
 		(property "Reference" "R701"
-			(at -1.235559 0.653823 0)
+			(at 4.37 0.05 0)
 			(unlocked yes)
 			(layer "B.SilkS")
@@
 		(tags "resistor")
 		(property "Reference" "R879"
-			(at 0 2.62 90)
+			(at -0.06 -2.99 90)
 			(layer "B.SilkS")
 			(effects
@@
 		(at 197.042 72.891 180)
 		(property "Reference" "R868"
-			(at -2 0.5 180)
+			(at 7.272 0.281 180)
 			(unlocked yes)
 			(layer "B.SilkS")
@@
 		(at 165.78 43.67 180)
 		(property "Reference" "R905"
-			(at -1.5 -1.64 0)
+			(at -1.74 1.15 0)
 			(unlocked yes)
 			(layer "B.SilkS")
@@
 		(tags "fuse")
 		(property "Reference" "F851"
-			(at 0 1.43 0)
+			(at -5.52 -0.27 0)
 			(layer "B.SilkS")
 			(effects
@@
 		(tags "fuse")
 		(property "Reference" "F849"
-			(at 3.5 0 0)
+			(at 6.345 -0.0325 0)
 			(layer "B.SilkS")
 			(effects
@@
 		(at 197.1525 58.4625 180)
 		(property "Reference" "R869"
-			(at -2 0.5 180)
+			(at 6.9625 0.7225 180)
 			(unlocked yes)
 			(layer "B.SilkS")
@@
 		(at 142.89 71.9 180)
 		(property "Reference" "R900"
-			(at -1.235559 0.653823 0)
+			(at -1.14 0.78 0)
 			(unlocked yes)
 			(layer "B.SilkS")
@@
 		(at 118.356 74.531928)
 		(property "Reference" "R318"
-			(at -1.235559 0.653823 180)
+			(at -1.316 -3.341928 180)
 			(unlocked yes)
 			(layer "B.SilkS")
@@
 		(at 175.04 45.23 180)
 		(property "Reference" "R700"
-			(at -1.235559 0.653823 0)
+			(at -7.21 -0.52 0)
 			(unlocked yes)
 			(layer "B.SilkS")
@@
 		(at 175.22 57.945 180)
 		(property "Reference" "R867"
-			(at -2 0.5 180)
+			(at -4.54 0.725 180)
 			(unlocked yes)
 			(layer "B.SilkS")
@@
 		(at 175.58 31.49 180)
 		(property "Reference" "R873"
-			(at -1.5 0.5 180)
+			(at -4.07 0.46 180)
 			(unlocked yes)
 			(layer "B.SilkS")
@@
 		(at 118.322 73.009)
 		(property "Reference" "R319"
-			(at -1.235559 0.653823 180)
+			(at -1.262 -3.059 180)
 			(unlocked yes)
 			(layer "B.SilkS")
@@
 		(at 142.36 29.26 180)
 		(property "Reference" "R903"
-			(at -1.235559 0.653823 0)
+			(at -1.37 1.65 0)
 			(unlocked yes)
 			(layer "B.SilkS")
@@
 		(at 56.335 21.807928)
 		(property "Reference" "R323"
-			(at -1.235559 0.653823 180)
+			(at -1.505 -3.307928 180)
 			(unlocked yes)
 			(layer "B.SilkS")
@@
 		(tags "resistor")
 		(property "Reference" "R870"
-			(at 0.0375 4 90)
+			(at -0.23 -2.94 90)
 			(layer "B.SilkS")
 			(effects
@@
 		(at 143.13 56.43 180)
 		(property "Reference" "R901"
-			(at -1.235559 0.653823 0)
+			(at -1.25 0.82 0)
 			(unlocked yes)
 			(layer "B.SilkS")
@@
 		(tags "SOD-123")
 		(property "Reference" "D844"
-			(at 0 2 0)
+			(at -0.348 -1.922 0)
 			(layer "B.SilkS")
 			(effects
@@
 		(tags "fuse")
 		(property "Reference" "F847"
-			(at 3.5 0 0)
+			(at 5.29 0.2 0)
 			(layer "B.SilkS")
 			(effects
@@
 		(tags "resistor")
 		(property "Reference" "R876"
-			(at 0 3 90)
+			(at 0.255 -3.185 90)
 			(layer "B.SilkS")
 			(effects
@@
 		(tags "SOD-123")
 		(property "Reference" "D842"
-			(at 0 2 0)
+			(at -0.482 -1.717 0)
 			(layer "B.SilkS")
 			(effects
@@
 		(at 56.291 24.586928)
 		(property "Reference" "R321"
-			(at -1.235559 0.653823 180)
+			(at -1.531 2.453072 180)
 			(unlocked yes)
 			(layer "B.SilkS")
@@
 		(tags "fuse")
 		(property "Reference" "F845"
-			(at 3.5 0 0)
+			(at 3.611 -0.266 0)
 			(layer "B.SilkS")
 			(effects
@@
 		(tags "fuse")
 		(property "Reference" "F844"
-			(at 3.5 0 0)
+			(at 6.19 0.175 0)
 			(layer "B.SilkS")
 			(effects
@@
 		(tags "fuse")
 		(property "Reference" "F848"
-			(at 3.5 0 0)
+			(at -4.3675 -0.7825 0)
 			(layer "B.SilkS")
 			(effects
@@
 		(at 142.31 43.54 180)
 		(property "Reference" "R902"
-			(at -1.235559 0.653823 0)
+			(at -1.4 1.19 0)
 			(unlocked yes)
 			(layer "B.SilkS")
@@
 		(tags "fuse")
 		(property "Reference" "F850"
-			(at 0 1.43 0)
+			(at 5.55 -0.14 0)
 			(layer "B.SilkS")
 			(effects
@@
 		(at 56.276 25.98)
 		(property "Reference" "R320"
-			(at -1.235559 0.653823 180)
+			(at -1.606 2.23 180)
 			(unlocked yes)
 			(layer "B.SilkS")
@@
 		(at 56.321 23.201)
 		(property "Reference" "R322"
-			(at -1.235559 0.653823 180)
+			(at -1.181 -3.451 180)
 			(unlocked yes)
 			(layer "B.SilkS")
@@
 		(at 197.115 45.595 180)
 		(property "Reference" "R874"
-			(at -1.5 0.5 180)
+			(at 7.005 0.895 180)
 			(unlocked yes)
 			(layer "B.SilkS")
@@
 		(at 166.1 30.01 180)
 		(property "Reference" "R904"
-			(at -1.235559 0.653823 0)
+			(at -1.62 1.69 0)
 			(unlocked yes)
 			(layer "B.SilkS")
@@
 		(tags "fuse")
 		(property "Reference" "F846"
-			(at 3.5 0 0)
+			(at -5.11 -0.22 0)
 			(layer "B.SilkS")
 			(effects
@@
 		(at 118.322 77.406928)
 		(property "Reference" "R316"
-			(at -1.235559 0.653823 180)
+			(at -1.422 2.243072 180)
 			(unlocked yes)
 			(layer "B.SilkS")
@@
 		(at 118.293 75.962)
 		(property "Reference" "R317"
-			(at -1.235559 0.653823 180)
+			(at -1.413 2.378 180)
 			(unlocked yes)
 			(layer "B.SilkS")
@@
 		(at 175.335 74.0125 180)
 		(property "Reference" "R875"
-			(at -1.5 0.5 180)
+			(at -4.135 0.5625 180)
 			(unlocked yes)
 			(layer "B.SilkS")
