File: greenenergyecu.kicad_sch (KiCad schematic)
At the start: 1 part, among them U1 ICM7555xB

Commit message: rt
Parts:
- removed U1: ICM7555xB, Package_SO:SOIC-8_3.9x4.9mm_P1.27mm, symbol Timer:ICM7555xB
- added M1: Module-knock-0.2, hellen-one-knock-0.2:knock, symbol knock:Module-knock-0.2
Changed lines of the file:
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@@
 	(generator_version "8.0")
 	(paper "A4")
-	(wire
-		(pts
-			(xy 82.55 82.55) (xy 78.74 82.55)
-		)
-		(stroke
-			(width 0)
-			(type default)
-		)
-	)
-	(wire
-		(pts
-			(xy 78.74 82.55) (xy 78.74 97.79)
-		)
-		(stroke
-			(width 0)
-			(type default)
-		)
-	)
-	(wire
-		(pts
-			(xy 95.25 97.79) (xy 78.74 97.79)
-		)
-		(stroke
-			(width 0)
-			(type default)
-		)
-	)
 	(symbol
-		(lib_id "Timer:ICM7555xB")
-		(at 95.25 87.63 0)
+		(lib_id "knock:Module-knock-0.2")
+		(at 66.04 86.36 0)
 		(unit 1)
 		(exclude_from_sim no)
@@
 		(dnp no)
 		(fields_autoplaced yes)
-		(property "Reference" "U1"
-			(at 97.4441 74.93 0)
+		(property "Reference" "M1"
+			(at 109.22 90.2014 0)
 			(effects
 				(font
 					(size 1.27 1.27)
 				)
-				(justify left)
 			)
 		)
-		(property "Value" "ICM7555xB"
-			(at 97.4441 77.47 0)
+		(property "Value" "Module-knock-0.2"
+			(at 109.22 92.7414 0)
 			(effects
 				(font
 					(size 1.27 1.27)
 				)
-				(justify left)
 			)
 		)
-		(property "Footprint" "Package_SO:SOIC-8_3.9x4.9mm_P1.27mm"
-			(at 116.84 97.79 0)
+		(property "Footprint" "hellen-one-knock-0.2:knock"
+			(at 66.04 86.36 0)
 			(effects
 				(font
@@
 			)
 		)
-		(property "Datasheet" "http://www.intersil.com/content/dam/Intersil/documents/icm7/icm7555-56.pdf"
-			(at 116.84 97.79 0)
+		(property "Datasheet" ""
+			(at 66.04 86.36 0)
 			(effects
 				(font
@@
 			)
 		)
-		(property "Description" "CMOS General Purpose Timer, 555 compatible, SOIC-8"
-			(at 95.25 87.63 0)
+		(property "Description" "Hellen-One Knock Pre-amplifier Module"
+			(at 66.04 86.36 0)
 			(effects
 				(font
@@
 			)
 		)
-		(pin "4"
+		(pin "W1"
 		)
-		(pin "2"
+		(pin "W2"
 		)
-		(pin "5"
+		(pin "E1"
 		)
-		(pin "3"
+		(pin "E2"
 		)
-		(pin "8"
-		)
-		(pin "7"
-		)
-		(pin "6"
-		)
-		(pin "1"
+		(pin "E3"
 		)
 		(instances
 			(project ""
 				(path "/e34f8548-18bd-4553-87dc-fac974a7531b"
-					(reference "U1")
+					(reference "M1")
 					(unit 1)
 				)

Commit message: ee
Changed lines of the file:
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@@
 	(symbol
 		(lib_id "knock:Module-knock-0.2")
-		(at 66.04 86.36 0)
+		(at 80.01 64.77 0)
 		(unit 1)
 		(exclude_from_sim no)
@@
 		(fields_autoplaced yes)
 		(property "Reference" "M1"
-			(at 109.22 90.2014 0)
+			(at 123.19 68.6114 0)
 			(effects
 				(font
@@
 		)
 		(property "Value" "Module-knock-0.2"
-			(at 109.22 92.7414 0)
+			(at 123.19 71.1514 0)
 			(effects
 				(font
@@
 		)
 		(property "Footprint" "hellen-one-knock-0.2:knock"
-			(at 66.04 86.36 0)
+			(at 80.01 64.77 0)
 			(effects
 				(font
@@
 		)
 		(property "Datasheet" ""
-			(at 66.04 86.36 0)
+			(at 80.01 64.77 0)
 			(effects
 				(font
@@
 		)
 		(property "Description" "Hellen-One Knock Pre-amplifier Module"
-			(at 66.04 86.36 0)
+			(at 80.01 64.77 0)
 			(effects
 				(font
@@
 			)
 		)
+		(pin "W2"
+		)
+		(pin "E3"
+		)
 		(pin "W1"
-		)
-		(pin "W2"
 		)
 		(pin "E1"
@@
 		(pin "E2"
 		)
-		(pin "E3"
-		)
 		(instances

Commit message: ee
Parts:
- added M2: Module-wbo-0.5, hellen-one-wbo-0.5:wbo, symbol wbo:Module-wbo-0.5
Changed lines of the file:
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@@
 	(paper "A4")
+	(symbol
+		(lib_id "wbo:Module-wbo-0.5")
+		(at 170.18 46.99 0)
+		(unit 1)
+		(exclude_from_sim no)
+		(in_bom yes)
+		(on_board yes)
+		(dnp no)
+		(fields_autoplaced yes)
+		(property "Reference" "M2"
+			(at 186.69 41.91 0)
+			(effects
+				(font
+					(size 1.27 1.27)
+				)
+			)
+		)
+		(property "Value" "Module-wbo-0.5"
+			(at 186.69 44.45 0)
+			(effects
+				(font
+					(size 1.27 1.27)
+				)
+			)
+		)
+		(property "Footprint" "hellen-one-wbo-0.5:wbo"
+			(at 195.58 45.72 0)
+			(effects
+				(font
+					(size 1.27 1.27)
+				)
+				(hide yes)
+			)
+		)
+		(property "Datasheet" ""
+			(at 170.18 46.99 0)
+			(effects
+				(font
+					(size 1.27 1.27)
+				)
+				(hide yes)
+			)
+		)
+		(property "Description" ""
+			(at 170.18 46.99 0)
+			(effects
+				(font
+					(size 1.27 1.27)
+				)
+				(hide yes)
+			)
+		)
+		(pin "W8"
+		)
+		(pin "W3"
+		)
+		(pin "J1"
+		)
+		(pin "W6"
+		)
+		(pin "W4"
+		)
+		(pin "J_VCC2"
+		)
+		(pin "W7"
+		)
+		(pin "W1"
+		)
+		(pin "W5"
+		)
+		(pin "E4"
+		)
+		(pin "E1"
+		)
+		(pin "E5"
+		)
+		(pin "E6"
+		)
+		(pin "J_GND1"
+		)
+		(pin "J_GND2"
+		)
+		(pin "W2"
+		)
+		(pin "J_VCC1"
+		)
+		(pin "G"
+		)
+		(pin "W9"
+		)
+		(pin "E2"
+		)
+		(pin "J2"
+		)
+		(pin "E3"
+		)
+		(instances
+			(project ""
+				(path "/e34f8548-18bd-4553-87dc-fac974a7531b"
+					(reference "M2")
+					(unit 1)
+				)
+			)
+		)
+	)
 	(symbol
 		(lib_id "knock:Module-knock-0.2")

Commit message: ee
Parts:
- removed M2: Module-wbo-0.5, hellen-one-wbo-0.5:wbo, symbol wbo:Module-wbo-0.5
Changed lines of the file:
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@@
 	(paper "A4")
-	(symbol
-		(lib_id "wbo:Module-wbo-0.5")
-		(at 170.18 46.99 0)
-		(unit 1)
-		(exclude_from_sim no)
-		(in_bom yes)
-		(on_board yes)
-		(dnp no)
-		(fields_autoplaced yes)
-		(property "Reference" "M2"
-			(at 186.69 41.91 0)
-			(effects
-				(font
-					(size 1.27 1.27)
-				)
-			)
-		)
-		(property "Value" "Module-wbo-0.5"
-			(at 186.69 44.45 0)
-			(effects
-				(font
-					(size 1.27 1.27)
-				)
-			)
-		)
-		(property "Footprint" "hellen-one-wbo-0.5:wbo"
-			(at 195.58 45.72 0)
-			(effects
-				(font
-					(size 1.27 1.27)
-				)
-				(hide yes)
-			)
-		)
-		(property "Datasheet" ""
-			(at 170.18 46.99 0)
-			(effects
-				(font
-					(size 1.27 1.27)
-				)
-				(hide yes)
-			)
-		)
-		(property "Description" ""
-			(at 170.18 46.99 0)
-			(effects
-				(font
-					(size 1.27 1.27)
-				)
-				(hide yes)
-			)
-		)
-		(pin "W8"
-		)
-		(pin "W3"
-		)
-		(pin "J1"
-		)
-		(pin "W6"
-		)
-		(pin "W4"
-		)
-		(pin "J_VCC2"
-		)
-		(pin "W7"
-		)
-		(pin "W1"
-		)
-		(pin "W5"
-		)
-		(pin "E4"
-		)
-		(pin "E1"
-		)
-		(pin "E5"
-		)
-		(pin "E6"
-		)
-		(pin "J_GND1"
-		)
-		(pin "J_GND2"
-		)
-		(pin "W2"
-		)
-		(pin "J_VCC1"
-		)
-		(pin "G"
-		)
-		(pin "W9"
-		)
-		(pin "E2"
-		)
-		(pin "J2"
-		)
-		(pin "E3"
-		)
-		(instances
-			(project ""
-				(path "/e34f8548-18bd-4553-87dc-fac974a7531b"
-					(reference "M2")
-					(unit 1)
-				)
-			)
-		)
-	)
 	(symbol
 		(lib_id "knock:Module-knock-0.2")
@@
 					(size 1.27 1.27)
 				)
+				(hide yes)
 			)
 		)

Commit message: ee
Parts:
- added M2: Module-wbo-0.5, hellen-one-wbo-0.5:wbo, symbol wbo:Module-wbo-0.5
Changed lines of the file:
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@@
 	(paper "A4")
+	(symbol
+		(lib_id "wbo:Module-wbo-0.5")
+		(at 41.91 105.41 0)
+		(unit 1)
+		(exclude_from_sim no)
+		(in_bom yes)
+		(on_board yes)
+		(dnp no)
+		(fields_autoplaced yes)
+		(property "Reference" "M2"
+			(at 58.42 100.33 0)
+			(effects
+				(font
+					(size 1.27 1.27)
+				)
+			)
+		)
+		(property "Value" "Module-wbo-0.5"
+			(at 58.42 102.87 0)
+			(effects
+				(font
+					(size 1.27 1.27)
+				)
+			)
+		)
+		(property "Footprint" "hellen-one-wbo-0.5:wbo"
+			(at 67.31 104.14 0)
+			(effects
+				(font
+					(size 1.27 1.27)
+				)
+				(hide yes)
+			)
+		)
+		(property "Datasheet" ""
+			(at 41.91 105.41 0)
+			(effects
+				(font
+					(size 1.27 1.27)
+				)
+				(hide yes)
+			)
+		)
+		(property "Description" ""
+			(at 41.91 105.41 0)
+			(effects
+				(font
+					(size 1.27 1.27)
+				)
+				(hide yes)
+			)
+		)
+		(pin "J2"
+		)
+		(pin "W6"
+		)
+		(pin "W9"
+		)
+		(pin "J_GND1"
+		)
+		(pin "W4"
+		)
+		(pin "J_GND2"
+		)
+		(pin "W8"
+		)
+		(pin "W5"
+		)
+		(pin "G"
+		)
+		(pin "J_VCC1"
+		)
+		(pin "W7"
+		)
+		(pin "E3"
+		)
+		(pin "W1"
+		)
+		(pin "W3"
+		)
+		(pin "E1"
+		)
+		(pin "E6"
+		)
+		(pin "E5"
+		)
+		(pin "J_VCC2"
+		)
+		(pin "J1"
+		)
+		(pin "E4"
+		)
+		(pin "W2"
+		)
+		(pin "E2"
+		)
+		(instances
+			(project ""
+				(path "/e34f8548-18bd-4553-87dc-fac974a7531b"
+					(reference "M2")
+					(unit 1)
+				)
+			)
+		)
+	)
 	(symbol
 		(lib_id "knock:Module-knock-0.2")

Commit message: wewe
Parts:
- removed M1: Module-knock-0.2, hellen-one-knock-0.2:knock, symbol knock:Module-knock-0.2
- removed M2: Module-wbo-0.5, hellen-one-wbo-0.5:wbo, symbol wbo:Module-wbo-0.5
- added D1, D2, D3, D4: B5819W, hellen-one-common:SOD-123, symbol hellen-one-common:1N4148WS
- added D5: SS34, Diode_SMD:D_SMA, symbol Diode:SS34
- added F1, F2, F3: 12H1500D, hellen-one-common:PAD-1206-PAD, symbol hellen-one-common:Fuse-Pad-Pad
- added J21: Conn_01x05_Male, Connector_Molex:Molex_SPOX_5267-05A_1x05_P2.50mm_Vertical, symbol Connector:Conn_01x05_Pin
- added J22: USB_B_Mini, hellen-one-common:USB-MINI-B-VERTICAL, symbol hellen-one-common:USB_B_Mini
- added M1: Module-power_12and5V-0.3, hellen-one-power_12and5V-0.3:power_12and5V, symbol hellen-one-power_12and5V:Module-power_12and5V-0.3
- added M2: Module-knock-0.2, hellen-one-knock-0.2:knock, symbol hellen-one-knock-0.2:Module-knock-0.2
- added M3: Module-vr-discrete-0.5, hellen-one-vr-discrete-0.5:vr-discrete, symbol hellen-one-vr-discrete-0.5:Module-vr-discrete-0.5
- added M4: Module-vr-max9924-0.1, hellen-one-vr-max9924-0.1:vr-max9924, symbol vr-max9924:Module-vr-max9924-0.1
- added M5: Module-wbo-0.5, hellen-one-wbo-0.5:wbo, symbol hellen-one-wbo-0.5:Module-wbo-0.5
- added M6: Module:mega-mcu100/0.3, hellen-one-mega-mcu100-0.3:mega-mcu100, symbol hellen-one-mega-mcu100-0.3:Module{colon}mega-mcu100/0.3
- added M7: Module-can-0.1, hellen-one-can-0.1:can, symbol hellen-one-can-0.1:Module-can-0.1
- added M8: Module-motor-driver-0.1, hellen-one-motor-driver-0.1:motor-driver, symbol motor-driver:Module-motor-driver-0.1
- added P1: 368255-2, 368255-2:368255-2, symbol 368255-2:368255-2
- added Q7: AO3400A, Package_TO_SOT_SMD:SOT-23, symbol Transistor_FET:AO3400A
- added R1, R15: 4.7k, hellen-one-common:R0603, symbol hellen-one-common:Res
- added R10, R11, R12: 10k, hellen-one-common:R0805, symbol hellen-one-common:Res
- added R2: 33k, hellen-one-common:R0603, symbol hellen-one-common:Res
- added R3: 6.8k, hellen-one-common:R0603, symbol hellen-one-common:Res
- added R4: Jumper-Pad-Pad, hellen-one-common:PAD-0805-PAD, symbol hellen-one-common:Jumper-Pad-Pad
- added R5, R6: 0, hellen-one-common:R0603, symbol hellen-one-common:Res
- added R54: 1k, hellen-one-common:R0603, symbol hellen-one-common:Res
- added R7, R8, R9: DNP, hellen-one-common:R0805, symbol hellen-one-common:Res
- added U10: BTS6143D, Package_TO_SOT_SMD:TO-252-4, symbol Power_Management:BTS6143D
Connections:
- new net: F3.2, M8.N2 (12V_IN), M8.S1 (12V_IN)
- new net: M1.E6 (PG_5VP), R4.1
- new net: M6.N14a (LED_GREEN), Q7.1 (G), R15.1
- new net: Q7.3 (D), U10.2 (IN)
- new net: R54.1, U10.4 (IS)
- new net: M5.J1 (SEL1), M5.J_GND1 (PULL_DOWN1)
- new net +12V: F2.1, F3.1, P1.120, P1.23, P1.24, R2.2, U10.3 (Vbb)
- new net +12V_PERM: M1.V1 (V12_PERM), P1.116
- new net +12V_RAW: D1.1 (K), D2.1 (K), D3.1 (K), D4.1 (K), F2.2, M1.V3 (V12_RAW), P1.117
- new net +3.3V: M6.N21 (V33), M8.W5 (3V3_IN)
- new net +3.3VA: M6.N15 (V33_SWITCHABLE), M7.V2 (CAN_VIO)
- new net +5V: M1.E4 (V5), M6.N22 (VCC)
- new net +5VA: M2.E1 (V5A), M3.E4 (V5_IN), M4.E4 (V5_IN), M5.W1 (V5_IN), M6.E1 (V5A_SWITCHABLE), M6.W2 (V5A_SWITCHABLE), M7.V1 (V5), R7.2, R8.2, R9.2
- new net +5VP: M1.V4 (5VP), P1.106, P1.107, P1.71, P1.72, P1.73, P1.74, P1.75, P1.76, P1.77, P1.78, P1.79, P1.80, R1.1
- new net ADC3: M6.S15 (IN_KNOCK_(PA2)), R5.2, R6.2
- new net DC1_DIR: M6.E21 (OUT_PWM4_(PC8)), M8.W4 (DIR)
- new net DC1_DIS_W1: M6.E8 (SPI2_MISO_(PB14)), M8.W1 (DIS)
- new net DC1_PWM: M6.E20 (OUT_PWM3_(PC7)), M8.W2 (PWM)
- new net DC2_DIR: M6.E9 (SPI2_MOSI_(PB15))
- new net DC2_DIS: M6.N4 (USBID_(PA10))
- new net DC2_PWM: M6.E22 (OUT_PWM5_(PC9))
- new net E6INJ7CANRX: M6.E6 (SPI2_CS_/_CAN2_RX_(PB12)), M7.V6 (CAN_RX)
- new net E7INJ8CANTX: M6.E7 (SPI2_SCK_/_CAN2_TX_(PB13)), M7.V5 (CAN_TX)
- new net EGT/SPI_CS: M6.N9 (SPI3_CS_(PA15))
- new net GND: D5.2 (A), J21.4 (Pin_4), J21.5 (Pin_5), J22.5 (GND), J22.6 (Shield), M1.S1 (GND), M2.E2 (GND), M3.G (GND), M4.G (GND), M5.E6 (LSU_H-), M5.G (GND), M6.G (GND), M7.E1 (GND), M8.G (GND), P1.114, P1.115, P1.3, Q7.2 (S), R15.2, R3.1, R54.2
- new net GNDA: M6.W1 (GNDA), P1.113, P1.52, P1.53, P1.54, P1.55, P1.56, P1.57, P1.58, P1.59, P1.60, P1.61, P1.62, P1.64, P1.66, P1.68, P1.98, P1.99, R10.1, R11.1, R12.1
- new net IGN1: M6.W10 (IGN1_(PC13))
- new net IGN2: M6.W9 (IGN2_(PE5))
- new net IGN3: M6.W8 (IGN3_(PE4))
- new net IGN4: M6.W7 (IGN4_(PE3))
- new net IGN5: M6.W6 (IGN5_(PE2))
- new net IGN6: M6.W5 (IGN6_(PB8))
- new net INJ1: M6.E17 (OUT_INJ1_(PD3))
- new net INJ2: M6.E16 (OUT_INJ2_(PA9))
- new net INJ3: M6.E15 (OUT_INJ3_(PD11))
- new net INJ4: M6.E14 (OUT_INJ4_(PD10))
- new net INJ5: M6.E13 (OUT_INJ5_(PD2))
- new net INJ6: M6.E12 (OUT_INJ6_(PA8))
- new net INTERNAL_MAP: M6.S12 (IN_MAP2_(PC1))
- new net IN_AUX3: M6.S7 (IN_AUX3_(PA7))
- new net IN_KNOCK: M2.E3 (OUT_KNOCK), R5.1
- new net IN_VIGN: F1.2, M1.V2 (IN_VIGN)
- new net IN_VMAIN: M6.S6 (IN_AUX4_(PC5)), R2.1, R3.2
- new net LS1: M6.E11 (OUT_INJ7_(PD15))
- new net LS2: M6.E10 (OUT_INJ8_(PD12))
- new net LS3: M6.E18 (OUT_PWM1_(PD13))
- new net LS4: M6.E19 (OUT_PWM2_(PC6))
- new net LS_HOT1: M6.W4 (IGN7_(PB9))
- new net LS_HOT2: M6.W3 (IGN8_(PE6))
- new net MISO3: M6.N11 (SPI3_MISO_(PC11))
- new net PG_5VP: M6.N12 (SPI3_MOSI_(PC12)), R4.2
- new net PIN1: M8.S3 (OUT+), P1.1
- new net PIN10: P1.10
- new net PIN100: P1.100
- new net PIN101: P1.101
- new net PIN102: M5.E4 (LSU_Rtrim), P1.102
- new net PIN103: M5.E3 (LSU_Ip), P1.103
- new net PIN104: M5.E2 (LSU_Vm), P1.104
- new net PIN105: M5.E1 (LSU_Un), P1.105
- new net PIN108: F1.1, P1.108
- new net PIN109: P1.109
- new net PIN11: P1.11
- new net PIN110: P1.110
- new net PIN111: P1.111
- new net PIN112: P1.112
- new net PIN118: P1.118
- new net PIN119: M5.E5 (LSU_H+), P1.119
- new net PIN12: P1.12
- new net PIN121: P1.121
- new net PIN13: P1.13
- new net PIN14: D1.2 (A), P1.14
- new net PIN15: D2.2 (A), P1.15
- new net PIN16: D3.2 (A), P1.16
- new net PIN17: M3.W2 (VR+), P1.17
- new net PIN18: M3.W1 (VR-), P1.18
- new net PIN19: M4.W2 (VR+), P1.19
- new net PIN2: M8.S2 (OUT-), P1.2
- new net PIN20: M4.W1 (VR-), P1.20, R1.2
- new net PIN21: P1.21
- new net PIN22: P1.22
- new net PIN25: P1.25
- new net PIN26: P1.26
- new net PIN27: P1.27
- new net PIN28: P1.28
- new net PIN29: P1.29
- new net PIN30: P1.30
- new net PIN31: P1.31
- new net PIN32: P1.32
- new net PIN33: P1.33
- new net PIN34: M6.S2 (IN_D3_(PE14)), P1.34
- new net PIN35: M6.S3 (IN_D2_(PE13)), P1.35
- new net PIN36: M6.S4 (IN_D1_(PE12)), P1.36
- new net PIN37: M6.S13 (IN_MAP1_(PC0)), P1.37
- new net PIN38: M6.S18 (IN_TPS_(PA4)), P1.38
- new net PIN39: M6.S9 (IN_AUX1_(PB0)), P1.39
- new net PIN4: P1.4
- new net PIN40: M6.S11 (IN_O2S_/_CAN_WAKEUP_(PA0)), P1.40
- new net PIN41: M6.S10 (IN_O2S2_(PA1)), P1.41
- new net PIN42: M6.S17 (IN_VSS_(PE11)), P1.42
- new net PIN43: D5.1 (K), P1.43, U10.1 (OUT), U10.5 (OUT)
- new net PIN44: P1.44
- new net PIN45: P1.45
- new net PIN46: P1.46
- new net PIN47: P1.47
- new net PIN48: P1.48
- new net PIN49: P1.49
- new net PIN5: P1.5
- new net PIN50: P1.50
- new net PIN51: P1.51
- new net PIN6: M6.N14 (UART2_RX_(PD6)), P1.6
- new net PIN63: M6.S20 (IN_IAT_(PC3)), P1.63
- new net PIN65: M6.S21 (IN_CLT_(PC2)), P1.65
- new net PIN67: P1.67
- new net PIN69: P1.69
- new net PIN7: M6.N13 (UART2_TX_(PD5)), P1.7
- new net PIN70: P1.70
- new net PIN8: P1.8
- new net PIN81: M2.W1 (IN_KNOCK), P1.81
- new net PIN82: M5.W4 (CANH), M6.W11 (CANH), P1.82
- new net PIN83: M5.W3 (CANL), M6.W12 (CANL), P1.83
- new net PIN84: M6.S14 (IN_CRANK_(PB1)), P1.84, R10.2, R7.1
- new net PIN85: M6.S16 (IN_CAM_(PA6)), P1.85, R11.2, R8.1
- new net PIN86: P1.86
- new net PIN87: P1.87
- new net PIN88: D4.2 (A), P1.88
- new net PIN89: M6.S1 (IN_D4_(PE15)), P1.89, R12.2, R9.1
- new net PIN9: P1.9
- new net PIN90: M6.S19 (IN_PPS_(PA3)), P1.90
- new net PIN91: M6.S8 (IN_AUX2_(PC4/PE9)), P1.91
- new net PIN92: P1.92
- new net PIN93: P1.93
- new net PIN94: P1.94
- new net PIN95: P1.95
- new net PIN96: P1.96
- new net PIN97: P1.97
- new net PWR_EN: M1.E5 (EN_5VP), M6.N20 (OUT_PWR_EN_(PE10))
- new net SCK3: M6.N10 (SPI3_SCK_(PC10))
- new net USB+: J21.3 (Pin_3), J22.3 (D+), M6.N3 (USBP_(PA12))
- new net USB-: J21.2 (Pin_2), J22.2 (D-), M6.N2 (USBM_(PA11))
- new net VBAT: M1.E1 (VBAT), M6.N17 (VBAT)
- new net VBUS: J21.1 (Pin_1), J22.1 (VBUS), M6.N1 (VBUS)
- new net VIGN: M1.E3 (VIGN), M6.E5 (IN_VIGN_(PA5))
- new net VREF1: M2.W2 (VREF), M6.S22 (VREF1)
- new net VR_DISCRETE: M3.E3 (OUT), M6.N18 (UART8_RX_(PE0))
- new net VR_DISCRETE_A: M3.E2 (OUT_A), R6.1
- new net VR_DISCRETE_THR: M3.E1 (Thresh_IN), M6.E23 (OUT_PWM6_(PD14))
- new net VR_MAX9924: M4.E3 (OUT), M6.N19 (UART8_TX_(PE1))
- no-connect marks 0 -> 22
Other:
- added sheet EGT (egt.kicad_sch)
- added sheet Ignition (IGN6.kicad_sch)
- added sheet Injector (INJ6.kicad_sch)
- added sheet LS (LS4.kicad_sch)
- added sheet LS HOT (LS_HOT.kicad_sch)
- note added: "#0"
- note added: "3.5A MAX Always hot capable"
- note added: "3.5A MAX Solenoid load capable"
- note added: "Analog inputs (sensors)"
- note added: "Bus types"
- note added: "Configurable "BUTTON" pulls"
- note added: "DC Motor"
- note added: "Discrete inputs"
- note added: "Flyback diodes"
- note added: "General purpose bus"
- note added: "Ignition"
- note added: "Injection"
- note added: "Install a 4.7 kOhm R1 resistor for using VR2- as a hall sensor input"
- note added: "LS & HS outputs"
- note added: "Move the resistor from position R143 to R145 to enable the CAN WAKEUP function. The AUX1 analog input will be unavailable."
- note added: "Move the resistor from position R6 to R5 to use ADC3 for receiving the analog signal VR-DISCRETE instead of the knock signal"
- note added: "Pin 8 may be used for shielding VR signals"
- note added: "Pin Name Recommended function B8 OUT_LS_HOT2 Fan Relay B9 OUT_LS_HOT1 Main Relay B16 OUT_LS4 Fuel Pump Replay B18 OUT_LS2 Idle Air Valve C8 GND VR Shield C15 IN_AUX3 Fuel Pressure D10 IN_BUTTON2 A/C Request All inputs are 12V-tolerant"
- company: (none) -> andreika @ rusEFI.comm
- title: (none) -> Hellen121vag

Commit message: w
Parts:
- R15: LCSC C21189 -> C23162
- R54: LCSC C21189 -> C21190
Changed lines of the file:
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@@
 			)
 		)
-		(property "LCSC" "C21189"
+		(property "LCSC" "C23162"
 			(at 388.62 227.33 0)
 			(effects
@@
 			)
 		)
-		(property "LCSC" "C21189"
+		(property "LCSC" "C21190"
 			(at 421.64 219.71 0)
 			(effects
