File: greenenergyecu.kicad_sch (KiCad schematic)
At the start: 35 parts, among them J21 Conn_01x05_Male, J22 USB_B_Mini, M1 Module-power_12and5V-0.3, M2 Module-knock-0.2, M3 Module-vr-discrete-0.5, M4 Module-vr-max9924-0.1, M5 Module-wbo-0.5, M6 Module:mega-mcu100/0.3, M7 Module-can-0.1, M8 Module-motor-driver-0.1, P1 368255-2, Q7 AO3400A, U10 BTS6143D

Commit message: weW
Parts:
- renumbered D5 to D1, D1 to D842, D2 to D843, D3 to D844, D4 to D845, F2 to F841, F1 to F842, F3 to F843, Q7 to Q1, R54 to R3, R15 to R4, R2 to R841, R3 to R842, R1 to R843, R4 to R846, R5 to R847, R6 to R848, U10 to U1
Connections:
- net PIN118 is gone; now on net LIBRE: P1.118
- net PIN121 is gone; now on net LIBRE: P1.121
- net PIN16 is gone; now on net OUT_LS2: D844.2 (A), P1.16
- net PIN25 is gone; now on net LIBRE: P1.25
- net PIN26 is gone; now on net LIBRE: P1.26
- net PIN29 is gone; now on net OUT_IGN4: P1.29
- net PIN30 is gone; now on net OUT_IGN3: P1.30
- net PIN31 is gone; now on net OUT_IGN2: P1.31
- net PIN32 is gone; now on net OUT_IGN1: P1.32
- net PIN67 is gone; now on net LIBRE: P1.67
- net PIN69 is gone; now on net LIBRE: P1.69
- net PIN70 is gone; now on net LIBRE: P1.70
- net PIN8 is gone; now on net OUT_IGN6: P1.8
- net PIN9 is gone; now on net OUT_IGN5: P1.9
- net PIN92 is gone; now on net LIBRE: P1.92
- net PIN93 is gone; now on net LIBRE: P1.93
- net PIN94 is gone; now on net LIBRE: P1.94
- net PIN95 is gone; now on net LIBRE: P1.95
- net PIN96 is gone; now on net LIBRE: P1.96
- net PIN97 is gone; now on net LIBRE: P1.97
- net USB+ is gone; now on net P_USB+: J21.3 (Pin_3), J22.3 (D+), M6.N3 (USBP_(PA12))
- net USB- is gone; now on net P_USB-: J21.2 (Pin_2), J22.2 (D-), M6.N2 (USBM_(PA11))
- net VBUS is gone; now on net P_VBUS: J21.1 (Pin_1), J22.1 (VBUS), M6.N1 (VBUS)
- net GND: now also P1.113
- net GNDA: no longer P1.113
- net PIN1 renamed OUT_DC1+
- net PIN10 renamed OUT_IGN4
- net PIN100 renamed WBO1_SWD
- net PIN101 renamed WBO1_SWC
- net PIN102 renamed 5_WBO_Rtrim
- net PIN103 renamed 1_WBO_Ip
- net PIN104 renamed 2_WBO_Vm
- net PIN105 renamed 6_WBO_Un
- net PIN108 renamed 12V_KEY
- net PIN109 renamed LIBRE
- net PIN11 renamed OUT_IGN3
- net PIN110 renamed P_VBUS
- net PIN111 renamed P_USB-
- net PIN112 renamed P_USB+
- net PIN119 renamed 3_WBO_Heater
- net PIN12 renamed OUT_IGN2
- net PIN13 renamed OUT_IGN1
- net PIN14 renamed OUT_LS1
- net PIN15 renamed OUT_LS2
- net PIN17 renamed VR_DISCRETE+
- net PIN18 renamed VR_DISCRETE-
- net PIN19 renamed VR_MAX9924+
- net PIN2 renamed OUT_DC1-
- net PIN20 renamed VR_MAX9924-
- net PIN21 renamed EGT+
- net PIN22 renamed EGT-
- net PIN27 renamed OUT_IGN6
- net PIN28 renamed OUT_IGN5
- net PIN33 renamed DIS
- net PIN34 renamed IN_HALL3
- net PIN35 renamed IN_HALL2
- net PIN36 renamed IN_HALL1
- net PIN37 renamed IN_MAP
- net PIN38 renamed IN_TPS1
- net PIN39 renamed IN_TPS2
- net PIN4 renamed OUT_DC2+
- net PIN40 renamed IN_AUX1
- net PIN41 renamed IN_AUX2
- net PIN42 renamed IN_FLEX
- net PIN43 renamed HSO
- net PIN44 renamed OUT_INJ1
- net PIN45 renamed OUT_INJ2
- net PIN46 renamed OUT_INJ3
- net PIN47 renamed OUT_INJ4
- net PIN48 renamed OUT_INJ5
- net PIN49 renamed OUT_INJ6
- net PIN5 renamed OUT_DC2-
- net PIN50 renamed OUT_INJ7
- net PIN51 renamed OUT_INJ8
- net PIN6 renamed UART_RX
- net PIN63 renamed IN_IAT
- net PIN65 renamed IN_CLT
- net PIN7 renamed UART_TX
- net PIN81 renamed IN_KNOCK_RAW
- net PIN82 renamed CAN+
- net PIN83 renamed CAN-
- net PIN84 renamed IN_BUTTON1
- net PIN85 renamed IN_BUTTON2
- net PIN86 renamed OUT_LS_HOT5
- net PIN87 renamed OUT_LS_HOT6
- net PIN88 renamed OUT_LS4
- net PIN89 renamed IN_BUTTON3
- net PIN90 renamed IN_PPS1
- net PIN91 renamed IN_PPS2
Other:
- moved on the sheet: J22

Commit message: weW
Parts:
- P1: footprint 368255-2:368255-2 -> footprints:368255-2
Changed lines of the file:
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@@
 			)
 		)
-		(property "Footprint" "368255-2:368255-2"
+		(property "Footprint" "footprints:368255-2"
 			(at 27.94 171.45 0)
 			(effects
@@
 			)
 		)
-		(property "Footprint" "368255-2:368255-2"
+		(property "Footprint" "footprints:368255-2"
 			(at 24.13 350.52 0)
 			(effects

Commit message: tilo
Parts:
- added R1: 1k, hellen-one-common:R0603, symbol hellen-one-common:Res
Connections:
- net GND: now also R1.2
Changed lines of the file:
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@@
 	)
 	(junction
+		(at 421.64 231.14)
+		(diameter 0)
+		(color 0 0 0 0)
+	)
+	(junction
 		(at 205.74 168.91)
 		(diameter 0)
@@
 		)
 	)
-	(wire
-		(pts
-			(xy 421.64 229.87) (xy 421.64 237.49)
-		)
-		(stroke
-			(width 0)
-			(type default)
-		)
-	)
 	(bus
 		(pts
@@
 	(wire
 		(pts
+			(xy 421.64 229.87) (xy 421.64 231.14)
+		)
+		(stroke
+			(width 0)
+			(type default)
+		)
+	)
+	(wire
+		(pts
 			(xy 252.73 257.81) (xy 262.89 257.81)
 		)
@@
 	(wire
 		(pts
+			(xy 421.64 231.14) (xy 421.64 237.49)
+		)
+		(stroke
+			(width 0)
+			(type default)
+		)
+	)
+	(wire
+		(pts
 			(xy 257.81 152.4) (xy 256.54 152.4)
 		)
@@
 	(wire
 		(pts
+			(xy 427.99 231.14) (xy 421.64 231.14)
+		)
+		(stroke
+			(width 0)
+			(type default)
+		)
+	)
+	(wire
+		(pts
 			(xy 129.54 196.85) (xy 120.65 196.85)
 		)
@@
 					(unit 1)
 				)
+			)
+		)
+	)
+	(symbol
+		(lib_id "hellen-one-common:Res")
+		(at 427.99 220.98 270)
+		(unit 1)
+		(exclude_from_sim no)
+		(in_bom yes)
+		(on_board yes)
+		(dnp no)
+		(property "Reference" "R1"
+			(at 430.53 226.06 0)
+			(effects
+				(font
+					(size 1.27 1.27)
+				)
+			)
+		)
+		(property "Value" "1k"
+			(at 427.99 226.06 0)
+			(effects
+				(font
+					(size 1.27 1.27)
+				)
+			)
+		)
+		(property "Footprint" "hellen-one-common:R0603"
+			(at 424.18 224.79 0)
+			(effects
+				(font
+					(size 1.27 1.27)
+				)
+				(hide yes)
+			)
+		)
+		(property "Datasheet" ""
+			(at 427.99 220.98 0)
+			(effects
+				(font
+					(size 1.27 1.27)
+				)
+				(hide yes)
+			)
+		)
+		(property "Description" ""
+			(at 427.99 220.98 0)
+			(effects
+				(font
+					(size 1.27 1.27)
+				)
+				(hide yes)
+			)
+		)
+		(property "LCSC" "C21190"
+			(at 427.99 220.98 0)
+			(effects
+				(font
+					(size 1.27 1.27)
+				)
+				(hide yes)
+			)
+		)
+		(property "comentario" ""
+			(at 427.99 220.98 0)
+			(effects
+				(font
+					(size 1.27 1.27)
+				)
+				(hide yes)
+			)
+		)
+		(pin "1"
+		)
+		(pin "2"
+		)
+		(instances
+			(project "greenenergyecu"
+				(path "/45c1f041-3b7c-4036-abe9-e26621c05a73"
+					(reference "R1")
+					(unit 1)
+				)

Commit message: tilo
Parts:
- removed J21: Conn_01x05_Male, Connector_Molex:Molex_SPOX_5267-05A_1x05_P2.50mm_Vertical, symbol Connector:Conn_01x05_Pin
- removed M7: Module-can-0.1, hellen-one-can-0.1:can, symbol hellen-one-can-0.1:Module-can-0.1
- removed R1: 1k, hellen-one-common:R0603, symbol hellen-one-common:Res
- added F1: 12H1500D, hellen-one-common:PAD-1206-PAD, symbol hellen-one-common:Fuse-Pad-Pad
- added M7: Module-can-0.1, hellen-one-can-0.1:can, symbol can:Module-can-0.1
Connections:
- net +12V: now also P1.3, P1.92, P1.93, P1.94, P1.95; no longer P1.120, P1.23, P1.24
- net +12V_PERM: now also P1.96, F1.1, F1.2; no longer P1.116
- net +12V_RAW: now also P1.63, P1.64; no longer P1.117
- net +3.3V: now also M7.V2 (CAN_VIO)
- net +5VA: now also M7.V1 (V5)
- net +5VP: now also P1.65, P1.66, P1.67, P1.68, P1.69, P1.70, P1.81; no longer P1.106, P1.107
- net 12V_KEY: now also P1.97; no longer P1.108
- net 1_WBO_Ip: now also P1.25; no longer P1.103
- net 2_WBO_Vm: now also P1.26; no longer P1.104
- net 3_WBO_Heater: now also P1.44, P1.45; no longer P1.119
- net 5_WBO_Rtrim: now also P1.6; no longer P1.102
- net 6_WBO_Un: now also P1.7; no longer P1.105
- net CAN+: no longer P1.82
- net CAN-: no longer P1.83
- net DIS: no longer P1.33
- net EGT+: no longer P1.21
- net EGT-: no longer P1.22
- net GND: now also P1.4, P1.5, P1.84, P1.85, P1.86, P1.87, P1.88, P1.89, M7.E1 (GND); no longer P1.113, P1.114, P1.115, P1.3
- net GNDA: now also P1.29, P1.46, P1.47, P1.48, P1.49, P1.50, P1.51; no longer P1.64, P1.66, P1.68, P1.98, P1.99
- net HSO: now also P1.1; no longer P1.43
- net INTERNAL_MAP: now also P1.20
- net IN_AUX1: now also P1.38; no longer P1.40
- net IN_AUX2: now also P1.19; no longer P1.41
- net IN_BUTTON1: no longer P1.84
- net IN_BUTTON2: no longer P1.85
- net IN_BUTTON3: no longer P1.89
- net IN_CLT: now also P1.23; no longer P1.65
- net IN_FLEX: now also P1.21; no longer P1.42
- net IN_HALL1: now also P1.17; no longer P1.36
- net IN_HALL2: now also P1.34; no longer P1.35
- net IN_HALL3: now also P1.15; no longer P1.34
- net IN_IAT: now also P1.41; no longer P1.63
- net IN_KNOCK_RAW: now also P1.10; no longer P1.81
- net IN_MAP: now also P1.39; no longer P1.37
- net IN_PPS1: now also P1.22; no longer P1.90
- net IN_PPS2: now also P1.18; no longer P1.91
- net IN_TPS1: now also P1.40; no longer P1.38
- net IN_TPS2: now also P1.37; no longer P1.39
- net LS2: now also M6.E19 (OUT_PWM2_(PC6)); no longer M6.E10 (OUT_INJ8_(PD12))
- net LS4: no longer M6.E19 (OUT_PWM2_(PC6))
- net OUT_DC1+: now also P1.90, P1.91; no longer M8.S3 (OUT+), P1.1
- net OUT_DC1-: now also P1.82, P1.83; no longer M8.S2 (OUT-), P1.2
- net OUT_DC2+: no longer P1.4
- net OUT_DC2-: no longer P1.5
- net OUT_IGN1: now also P1.114; no longer P1.13, P1.32
- net OUT_IGN2: now also P1.115; no longer P1.12, P1.31
- net OUT_IGN3: now also P1.116; no longer P1.11, P1.30
- net OUT_IGN4: now also P1.117; no longer P1.10, P1.29
- net OUT_IGN5: now also P1.118; no longer P1.28, P1.9
- net OUT_IGN6: now also P1.119; no longer P1.27, P1.8
- net OUT_INJ1: now also P1.106, P1.98; no longer P1.44
- net OUT_INJ2: now also P1.107, P1.99; no longer P1.45
- net OUT_INJ3: now also P1.100, P1.108; no longer P1.46
- net OUT_INJ4: now also P1.101, P1.109; no longer P1.47
- net OUT_INJ5: now also P1.102, P1.110; no longer P1.48
- net OUT_INJ6: now also P1.103, P1.111; no longer P1.49
- net OUT_INJ7: now also P1.104, P1.112; no longer P1.50
- net OUT_INJ8: now also P1.105, P1.113; no longer P1.51
- net OUT_LS1: now also P1.11; no longer P1.14
- net OUT_LS2: now also P1.30; no longer D844.2 (A), P1.15, P1.16
- net OUT_LS_HOT5: no longer P1.86
- net OUT_LS_HOT6: no longer P1.87
- net P_USB+: now also P1.33; no longer P1.112
- net P_USB-: now also P1.14; no longer P1.111
- net P_VBUS: now also P1.32; no longer P1.110
- net UART_RX: now also P1.16; no longer P1.6
- net UART_TX: now also P1.35; no longer P1.7
- net VR_DISCRETE+: now also P1.8; no longer P1.17
- net VR_DISCRETE-: now also P1.27; no longer P1.18
- net VR_MAX9924+: now also P1.9; no longer P1.19
- net VR_MAX9924-: now also P1.28; no longer P1.20, R843.2
- net WBO1_SWC: no longer P1.101
- net WBO1_SWD: no longer P1.100
- net at F843.2, M8.S1 (12V_IN): no longer M8.N2 (12V_IN)
- net E6INJ7CANRX: no longer names the net of M6.E6 (SPI2_CS_/_CAN2_RX_(PB12))
- net E6INJ7CANRX: now also M7.V6 (CAN_RX)
- net E7INJ8CANTX: no longer names the net of M6.E7 (SPI2_SCK_/_CAN2_TX_(PB13))
- net E7INJ8CANTX: now also M7.V5 (CAN_TX)
- net IN_AUX3 renamed AUX3
- net AUX3: now also P1.36
- removed net LIBRE: P1.109, P1.118, P1.121, P1.25, P1.26, P1.67, P1.69, P1.70, P1.92, P1.93, P1.94, P1.95, P1.96, P1.97
- net LS1 renamed INJ7
- net LS_HOT1 renamed IGN7
- net LS_HOT2 renamed IGN8
- net OUT_LS4 renamed FP_LS
- net FP_LS: no longer P1.88
- new net CAN_H: M7.S2 (CANH)
- new net CAN_L: M7.S1 (CANL)
- new net INJ8: M6.E10 (OUT_INJ8_(PD12))
- new net LSH/OUT1: P1.12
- new net LSH/OUT2: P1.13
- new net LSH/OUT3: P1.31
- new net MAIN_LS: D844.2 (A), P1.2
- new net OUT_IGN7: P1.120
- new net OUT_IGN8: P1.121
Other:
- removed sheet LS HOT
- added sheet LSH (LS_H.kicad_sch)
- sheet Ignition ports: added IN7, IN8, OUT7, OUT8; removed none
- sheet Injector ports: added 33v, 5v; removed none
- note removed: "3.5A MAX Always hot capable"
- moved on the sheet: R4
