File: greenenergyecu.kicad_sch (KiCad schematic)
At the start: 35 parts, among them J22 USB_B_Mini, M1 Module-power_12and5V-0.3, M2 Module-knock-0.2, M3 Module-vr-discrete-0.5, M4 Module-vr-max9924-0.1, M5 Module-wbo-0.5, M6 Module:mega-mcu100/0.3, M7 Module-can-0.1, M8 Module-motor-driver-0.1, P1 368255-2, Q1 AO3400A, U1 BTS6143D

Commit message: wew
Parts:
- P1: LCSC (none) -> C392284
Changed lines of the file:
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@@
+			)
+		)
+		(property "LCSC" "C392284"
+			(at 27.94 180.34 0)
+			(effects
+				(font
+					(size 1.27 1.27)
+				)
+				(hide yes)
 			)
 		)
@@
 			(at 27.94 356.87 0)
 			(effects
+				(font
+					(size 1.27 1.27)
+				)
+				(hide yes)
+			)
+		)
+		(property "LCSC" "C392284"
+			(at 27.94 356.87 0)
+			(effects

Commit message: ww
Parts:
- J22: LCSC (none) -> C2682228; MyComment DNP -> (none)
Changed lines of the file:
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@@
 			)
 		)
-		(property "LCSC" ""
+		(property "LCSC" "C2682228"
 			(at 394.97 302.26 0)
 			(effects
@@
 			)
 		)
-		(property "MyComment" "DNP"
+		(property "MyComment" ""
 			(at 400.05 311.785 0)
 			(effects

Commit message: ww
Parts:
- D1: LCSC (none) -> C5119706
- Q1: LCSC (none) -> C20917
- U1: LCSC (none) -> C95232
Changed lines of the file:
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@@
 			)
 		)
+		(property "LCSC" "C5119706"
+			(at 414.02 194.31 0)
+			(effects
+				(font
+					(size 1.27 1.27)
+				)
+				(hide yes)
+			)
+		)
 		(pin "2"
 		)
@@
 			)
 		)
+		(property "LCSC" "C20917"
+			(at 405.13 227.33 0)
+			(effects
+				(font
+					(size 1.27 1.27)
+				)
+				(hide yes)
+			)
+		)
 		(pin "2"
 		)
@@
 			(effects
 				(font
+					(size 1.27 1.27)
+				)
+				(hide yes)
+			)
+		)
+		(property "LCSC" "C95232"
+			(at 410.21 209.55 90)
+			(effects
+				(font

Commit message: w
Connections:
- net OUT_DC1+: now also P1.82, P1.83; no longer P1.90, P1.91
- net OUT_DC1-: now also P1.90, P1.91; no longer P1.82, P1.83

Commit message: w
Other:
- sheet LSH ports: added none; removed IN1, IN3, OUT1, OUT3
Changed lines of the file:
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@@
-			)
-		)
-		(pin "IN1" input
-			(at 97.79 298.45 0)
-			(effects
-				(font
-					(size 1.27 1.27)
-				)
-				(justify right)
-			)
-		)
-		(pin "OUT3" output
-			(at 85.09 303.53 180)
-			(effects
-				(font
-					(size 1.27 1.27)
-				)
-				(justify left)
-			)
-		)
-		(pin "OUT1" output
-			(at 85.09 298.45 180)
-			(effects
-				(font
-					(size 1.27 1.27)
-				)
-				(justify left)
 			)
 		)
@@
 			(effects
 				(font
-					(size 1.27 1.27)
-				)
-				(justify right)
-			)
-		)
-		(pin "IN3" input
-			(at 97.79 303.53 0)
-			(effects
-				(font

Commit message: a
Changed lines of the file:
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@@
+		)
+	)
+	(global_label "+12V_RAW"
+		(shape input)
+		(at 76.2 179.07 0)
+		(fields_autoplaced yes)
+		(effects
+			(font
+				(size 1.27 1.27)
+			)
+			(justify left)
+		)
+		(property "Intersheetrefs" "${INTERSHEET_REFS}"
+			(at 89.0428 179.07 0)
+			(effects
+				(font
+					(size 1.27 1.27)
+				)
+				(justify left)
+				(hide yes)
+			)
 		)
 	)

Commit message: weew
Changed lines of the file:
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@@
+	)
+	(symbol
+		(lib_name "LOGO_1")
+		(lib_id "lokon:LOGO")
+		(at 367.03 407.67 0)
+		(unit 1)
+		(exclude_from_sim no)
+		(in_bom yes)
+		(on_board yes)
+		(dnp no)
+		(fields_autoplaced yes)
+		(property "Reference" "#G2"
+			(at 367.03 405.5029 0)
+			(effects
+				(font
+					(size 1.27 1.27)
+				)
+				(hide yes)
+			)
+		)
+		(property "Value" "LOGO"
+			(at 367.03 409.8371 0)
+			(effects
+				(font
+					(size 1.27 1.27)
+				)
+				(hide yes)
+			)
+		)
+		(property "Footprint" ""
+			(at 367.03 407.67 0)
+			(effects
+				(font
+					(size 1.27 1.27)
+				)
+				(hide yes)
+			)
+		)
+		(property "Datasheet" ""
+			(at 367.03 407.67 0)
+			(effects
+				(font
+					(size 1.27 1.27)
+				)
+				(hide yes)
+			)
+		)
+		(property "Description" ""
+			(at 367.03 407.67 0)
+			(effects
+				(font
+					(size 1.27 1.27)
+				)
+				(hide yes)
+			)
+		)
+		(instances
+			(project ""
+				(path "/45c1f041-3b7c-4036-abe9-e26621c05a73"
+					(reference "#G2")
+					(unit 1)
+				)
+			)
+		)
 	)
 	(symbol
