File: LS4.kicad_sch (KiCad schematic)
At the start: 10 parts, among them U1 VNLD5160TR-E, U2 VNLD5160TR-E

Commit message: weW
Parts:
- renumbered U1 to U842, U2 to U843
Changed lines of the file:
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@@
 		(on_board yes)
 		(dnp no)
-		(property "Reference" "U2"
+		(property "Reference" "U843"
 			(at 146.05 95.25 0)
 			(effects
@@
 			(project "greenenergyecu"
 				(path "/45c1f041-3b7c-4036-abe9-e26621c05a73/37c68176-bc6d-4360-9788-c5c46985dc55"
-					(reference "U2")
+					(reference "U843")
 					(unit 1)
 				)
@@
 		(on_board yes)
 		(dnp no)
-		(property "Reference" "U1"
+		(property "Reference" "U842"
 			(at 143.51 55.88 0)
 			(effects
@@
 			(project "greenenergyecu"
 				(path "/45c1f041-3b7c-4036-abe9-e26621c05a73/37c68176-bc6d-4360-9788-c5c46985dc55"
-					(reference "U1")
-					(unit 1)
-				)
+					(reference "U842")
+					(unit 1)
+				)

Commit message: weW
Parts:
- renumbered R13 to R316, R16 to R317, R14 to R318, R17 to R319, R18 to R320, R20 to R321, R19 to R322, R21 to R323
Changed lines of the file:
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@@
 		(on_board yes)
 		(dnp no)
-		(property "Reference" "R20"
+		(property "Reference" "R321"
 			(at 182.88 95.25 0)
 			(effects
@@
 			(project "greenenergyecu"
 				(path "/45c1f041-3b7c-4036-abe9-e26621c05a73/37c68176-bc6d-4360-9788-c5c46985dc55"
-					(reference "R20")
+					(reference "R321")
 					(unit 1)
 				)
@@
 		(on_board yes)
 		(dnp no)
-		(property "Reference" "R21"
+		(property "Reference" "R323"
 			(at 182.88 113.03 0)
 			(effects
@@
 			(project "greenenergyecu"
 				(path "/45c1f041-3b7c-4036-abe9-e26621c05a73/37c68176-bc6d-4360-9788-c5c46985dc55"
-					(reference "R21")
+					(reference "R323")
 					(unit 1)
 				)
@@
 		(on_board yes)
 		(dnp no)
-		(property "Reference" "R17"
+		(property "Reference" "R319"
 			(at 173.99 73.66 0)
 			(effects
@@
 			(project "greenenergyecu"
 				(path "/45c1f041-3b7c-4036-abe9-e26621c05a73/37c68176-bc6d-4360-9788-c5c46985dc55"
-					(reference "R17")
+					(reference "R319")
 					(unit 1)
 				)
@@
 		(on_board yes)
 		(dnp no)
-		(property "Reference" "R19"
+		(property "Reference" "R322"
 			(at 177.8 105.41 0)
 			(effects
@@
 			(project "greenenergyecu"
 				(path "/45c1f041-3b7c-4036-abe9-e26621c05a73/37c68176-bc6d-4360-9788-c5c46985dc55"
-					(reference "R19")
+					(reference "R322")
 					(unit 1)
 				)
@@
 		(on_board yes)
 		(dnp no)
-		(property "Reference" "R13"
+		(property "Reference" "R316"
 			(at 170.18 60.96 0)
 			(effects
@@
 			(project "greenenergyecu"
 				(path "/45c1f041-3b7c-4036-abe9-e26621c05a73/37c68176-bc6d-4360-9788-c5c46985dc55"
-					(reference "R13")
+					(reference "R316")
 					(unit 1)
 				)
@@
 		(on_board yes)
 		(dnp no)
-		(property "Reference" "R14"
+		(property "Reference" "R318"
 			(at 170.18 66.04 0)
 			(effects
@@
 			(project "greenenergyecu"
 				(path "/45c1f041-3b7c-4036-abe9-e26621c05a73/37c68176-bc6d-4360-9788-c5c46985dc55"
-					(reference "R14")
+					(reference "R318")
 					(unit 1)
 				)
@@
 		(on_board yes)
 		(dnp no)
-		(property "Reference" "R18"
+		(property "Reference" "R320"
 			(at 177.8 100.33 0)
 			(effects
@@
 			(project "greenenergyecu"
 				(path "/45c1f041-3b7c-4036-abe9-e26621c05a73/37c68176-bc6d-4360-9788-c5c46985dc55"
-					(reference "R18")
+					(reference "R320")
 					(unit 1)
 				)
@@
 		(on_board yes)
 		(dnp no)
-		(property "Reference" "R16"
+		(property "Reference" "R317"
 			(at 173.99 58.42 0)
 			(effects
@@
 			(project "greenenergyecu"
 				(path "/45c1f041-3b7c-4036-abe9-e26621c05a73/37c68176-bc6d-4360-9788-c5c46985dc55"
-					(reference "R16")
-					(unit 1)
-				)
+					(reference "R317")
+					(unit 1)
+				)
