File: LS_HOT.kicad_sch (KiCad schematic)
At the start: 5 parts, among them U7 VNLD5160TR-E

Commit message: weW
Parts:
- renumbered U7 to U844
Changed lines of the file:
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@@
 		(dnp no)
 		(fields_autoplaced yes)
-		(property "Reference" "U7"
+		(property "Reference" "U844"
 			(at 125.73 73.66 0)
 			(effects
@@
 			(project "greenenergyecu"
 				(path "/45c1f041-3b7c-4036-abe9-e26621c05a73/bdc55f5a-1abb-4701-b1a5-3e8a3596401f"
-					(reference "U7")
+					(reference "U844")
 					(unit 1)
 				)

Commit message: weW
Parts:
- renumbered R50 to R300, R51 to R301, R52 to R302, R53 to R303
Changed lines of the file:
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@@
 		(on_board yes)
 		(dnp no)
-		(property "Reference" "R52"
+		(property "Reference" "R302"
 			(at 156.21 83.82 0)
 			(effects
@@
 			(project "greenenergyecu"
 				(path "/45c1f041-3b7c-4036-abe9-e26621c05a73/bdc55f5a-1abb-4701-b1a5-3e8a3596401f"
-					(reference "R52")
+					(reference "R302")
 					(unit 1)
 				)
@@
 		(on_board yes)
 		(dnp no)
-		(property "Reference" "R50"
+		(property "Reference" "R300"
 			(at 156.21 78.74 0)
 			(effects
@@
 			(project "greenenergyecu"
 				(path "/45c1f041-3b7c-4036-abe9-e26621c05a73/bdc55f5a-1abb-4701-b1a5-3e8a3596401f"
-					(reference "R50")
+					(reference "R300")
 					(unit 1)
 				)
@@
 		(on_board yes)
 		(dnp no)
-		(property "Reference" "R53"
+		(property "Reference" "R303"
 			(at 158.75 91.44 0)
 			(effects
@@
 			(project "greenenergyecu"
 				(path "/45c1f041-3b7c-4036-abe9-e26621c05a73/bdc55f5a-1abb-4701-b1a5-3e8a3596401f"
-					(reference "R53")
+					(reference "R303")
 					(unit 1)
 				)
@@
 		(on_board yes)
 		(dnp no)
-		(property "Reference" "R51"
+		(property "Reference" "R301"
 			(at 158.75 76.2 0)
 			(effects
@@
 			(project "greenenergyecu"
 				(path "/45c1f041-3b7c-4036-abe9-e26621c05a73/bdc55f5a-1abb-4701-b1a5-3e8a3596401f"
-					(reference "R51")
-					(unit 1)
-				)
+					(reference "R301")
+					(unit 1)
+				)
