File: egt.kicad_sch (KiCad schematic)
At the start: 9 parts, among them U8 MAX31855KASA

Commit message: weW
Parts:
- removed U8: MAX31855KASA, Package_SO:SOIC-8_3.9x4.9mm_P1.27mm, symbol Sensor_Temperature:MAX31855KASA
- added U846: MAX31855KASA, Package_SO:SOIC-8_3.9x4.9mm_P1.27mm, symbol Sensor_Temperature:MAX31855KASA
- renumbered C1 to C843, C3 to C844, C2 to C845, D6 to D846, L1 to L841, L2 to L842
Connections:
- net SPI_CS: now also U846.6 (~{CS})
- net SPI_SCK: now also U846.5 (SCK)
- net SPI_SO: now also U846.7 (SO)
- net Vcc: now also U846.4 (V_{CC})
- net at C843.2, C845.1, D846.1 (K)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: now also U846.2 (T-)
- net at C844.2, C845.2, D846.2 (K)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: now also U846.3 (T+)
Changed lines of the file:
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@@
+	)
+	(symbol
+		(lib_id "Sensor_Temperature:MAX31855KASA")
+		(at 160.02 87.63 0)
+		(unit 1)
+		(exclude_from_sim no)
+		(in_bom yes)
+		(on_board yes)
+		(dnp no)
+		(fields_autoplaced yes)
+		(property "Reference" "U846"
+			(at 162.2141 74.93 0)
+			(effects
+				(font
+					(size 1.27 1.27)
+				)
+				(justify left)
+			)
+		)
+		(property "Value" "MAX31855KASA"
+			(at 162.2141 77.47 0)
+			(effects
+				(font
+					(size 1.27 1.27)
+				)
+				(justify left)
+			)
+		)
+		(property "Footprint" "Package_SO:SOIC-8_3.9x4.9mm_P1.27mm"
+			(at 162.56 97.79 0)
+			(effects
+				(font
+					(size 1.27 1.27)
+					(italic yes)
+				)
+				(justify left)
+				(hide yes)
+			)
+		)
+		(property "Datasheet" "http://datasheets.maximintegrated.com/en/ds/MAX31855.pdf"
+			(at 162.56 100.33 0)
+			(effects
+				(font
+					(size 1.27 1.27)
+				)
+				(justify left)
+				(hide yes)
+			)
+		)
+		(property "Description" "Cold Junction K-type Thermocouple Interface, SPI, SOIC-8"
+			(at 162.56 95.25 0)
+			(effects
+				(font
+					(size 1.27 1.27)
+				)
+				(justify left)
+				(hide yes)
+			)
+		)
+		(pin "4"
+		)
+		(pin "3"
+		)
+		(pin "1"
+		)
+		(pin "8"
+		)
+		(pin "5"
+		)
+		(pin "6"
+		)
+		(pin "2"
+		)
+		(pin "7"
+		)
+		(instances
+			(project ""
+				(path "/45c1f041-3b7c-4036-abe9-e26621c05a73/6cde32b6-05f2-499d-9aff-ad44aab97055"
+					(reference "U846")
+					(unit 1)
+				)
+			)
+		)
 	)
 	(symbol
@@
 		(on_board yes)
 		(dnp no)
-		(property "Reference" "C2"
+		(property "Reference" "C845"
 			(at 138.43 84.455 90)
 			(effects
@@
 			(project "greenenergyecu"
 				(path "/45c1f041-3b7c-4036-abe9-e26621c05a73/6cde32b6-05f2-499d-9aff-ad44aab97055"
-					(reference "C2")
+					(reference "C845")
 					(unit 1)
 				)
@@
 		(on_board yes)
 		(dnp no)
-		(property "Reference" "C1"
+		(property "Reference" "C843"
 			(at 132.08 94.615 90)
 			(effects
@@
 			(project "greenenergyecu"
 				(path "/45c1f041-3b7c-4036-abe9-e26621c05a73/6cde32b6-05f2-499d-9aff-ad44aab97055"
-					(reference "C1")
+					(reference "C843")
 					(unit 1)
 				)
@@
 		(on_board yes)
 		(dnp no)
-		(property "Reference" "L1"
+		(property "Reference" "L841"
 			(at 100.33 85.09 90)
 			(effects
@@
 			(project "greenenergyecu"
 				(path "/45c1f041-3b7c-4036-abe9-e26621c05a73/6cde32b6-05f2-499d-9aff-ad44aab97055"
-					(reference "L1")
+					(reference "L841")
 					(unit 1)
 				)
@@
 		(on_board yes)
 		(dnp no)
-		(property "Reference" "D6"
+		(property "Reference" "D846"
 			(at 114.3 100.33 0)
 			(effects
@@
 			(project "greenenergyecu"
 				(path "/45c1f041-3b7c-4036-abe9-e26621c05a73/6cde32b6-05f2-499d-9aff-ad44aab97055"
-					(reference "D6")
+					(reference "D846")
 					(unit 1)
 				)
@@
 		(on_board yes)
 		(dnp no)
-		(property "Reference" "L2"
+		(property "Reference" "L842"
 			(at 100.33 92.71 90)
 			(effects
@@
 			(project "greenenergyecu"
 				(path "/45c1f041-3b7c-4036-abe9-e26621c05a73/6cde32b6-05f2-499d-9aff-ad44aab97055"
-					(reference "L2")
+					(reference "L842")
 					(unit 1)
 				)
@@
 		(on_board yes)
 		(dnp no)
-		(property "Reference" "C3"
+		(property "Reference" "C844"
 			(at 147.32 94.615 90)
 			(effects
@@
 			(project "greenenergyecu"
 				(path "/45c1f041-3b7c-4036-abe9-e26621c05a73/6cde32b6-05f2-499d-9aff-ad44aab97055"
-					(reference "C3")
-					(unit 1)
-				)
-			)
-		)
-	)
-	(symbol
-		(lib_name "MAX31855KASA_1")
-		(lib_id "Sensor_Temperature:MAX31855KASA")
-		(at 160.02 87.63 0)
-		(unit 1)
-		(exclude_from_sim no)
-		(in_bom yes)
-		(on_board yes)
-		(dnp no)
-		(property "Reference" "U8"
-			(at 162.2141 74.93 0)
-			(effects
-				(font
-					(size 1.27 1.27)
-				)
-				(justify left)
-			)
-		)
-		(property "Value" "MAX31855KASA"
-			(at 162.2141 77.47 0)
-			(effects
-				(font
-					(size 1.27 1.27)
-				)
-				(justify left)
-			)
-		)
-		(property "Footprint" "Package_SO:SOIC-8_3.9x4.9mm_P1.27mm"
-			(at 185.42 96.52 0)
-			(effects
-				(font
-					(size 1.27 1.27)
-					(italic yes)
-				)
-				(hide yes)
-			)
-		)
-		(property "Datasheet" "http://datasheets.maximintegrated.com/en/ds/MAX31855.pdf"
-			(at 160.02 87.63 0)
-			(effects
-				(font
-					(size 1.27 1.27)
-				)
-				(hide yes)
-			)
-		)
-		(property "Description" ""
-			(at 160.02 87.63 0)
-			(effects
-				(font
-					(size 1.27 1.27)
-				)
-				(hide yes)
-			)
-		)
-		(property "LCSC" "C52028"
-			(at 160.02 87.63 0)
-			(effects
-				(font
-					(size 1.27 1.27)
-				)
-				(hide yes)
-			)
-		)
-		(property "comentario" ""
-			(at 160.02 87.63 0)
-			(effects
-				(font
-					(size 1.27 1.27)
-				)
-				(hide yes)
-			)
-		)
-		(pin "1"
-		)
-		(pin "2"
-		)
-		(pin "3"
-		)
-		(pin "4"
-		)
-		(pin "5"
-		)
-		(pin "6"
-		)
-		(pin "7"
-		)
-		(instances
-			(project "greenenergyecu"
-				(path "/45c1f041-3b7c-4036-abe9-e26621c05a73/6cde32b6-05f2-499d-9aff-ad44aab97055"
-					(reference "U8")
-					(unit 1)
-				)
+					(reference "C844")
+					(unit 1)
+				)

Commit message: tilo
Connections:
- net GND: now also U846.1 (GND)
Changed lines of the file:
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@@
 	(wire
 		(pts
-			(xy 160.02 97.79) (xy 160.02 100.33)
+			(xy 160.02 95.25) (xy 160.02 100.33)
 		)
 		(stroke

Commit message: ww
Parts:
- U846: LCSC (none) -> C52028
Changed lines of the file:
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@@
+			)
+		)
+		(property "LCSC" "C52028"
+			(at 160.02 87.63 0)
+			(effects
+				(font
+					(size 1.27 1.27)
+				)
+				(hide yes)
 			)
 		)
