File: INJ6.kicad_sch (KiCad schematic)
At the start: 20 parts, among them U3 VNLD5160TR-E, U4 VNLD5160TR-E, U5 VNLD5160TR-E, U6 VNLD5160TR-E

Commit message: weW
Parts:
- renumbered U3 to U2, U6 to U847, U4 to U848, U5 to U849
Changed lines of the file:
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@@
 		(on_board yes)
 		(dnp no)
-		(property "Reference" "U6"
+		(property "Reference" "U847"
 			(at 125.73 29.21 0)
 			(effects
@@
 			(project "greenenergyecu"
 				(path "/45c1f041-3b7c-4036-abe9-e26621c05a73/5bf5a5f3-cb81-43b4-ad19-7826a949969c"
-					(reference "U6")
+					(reference "U847")
 					(unit 1)
 				)
@@
 		(on_board yes)
 		(dnp no)
-		(property "Reference" "U4"
+		(property "Reference" "U848"
 			(at 124.46 68.58 0)
 			(effects
@@
 			(project "greenenergyecu"
 				(path "/45c1f041-3b7c-4036-abe9-e26621c05a73/5bf5a5f3-cb81-43b4-ad19-7826a949969c"
-					(reference "U4")
+					(reference "U848")
 					(unit 1)
 				)
@@
 		(on_board yes)
 		(dnp no)
-		(property "Reference" "U5"
+		(property "Reference" "U849"
 			(at 124.46 107.95 0)
 			(effects
@@
 			(project "greenenergyecu"
 				(path "/45c1f041-3b7c-4036-abe9-e26621c05a73/5bf5a5f3-cb81-43b4-ad19-7826a949969c"
-					(reference "U5")
+					(reference "U849")
 					(unit 1)
 				)
@@
 		(on_board yes)
 		(dnp no)
-		(property "Reference" "U3"
+		(property "Reference" "U2"
 			(at 120.65 146.05 0)
 			(effects
@@
 			(project "greenenergyecu"
 				(path "/45c1f041-3b7c-4036-abe9-e26621c05a73/5bf5a5f3-cb81-43b4-ad19-7826a949969c"
-					(reference "U3")
-					(unit 1)
-				)
+					(reference "U2")
+					(unit 1)
+				)

Commit message: weW
Parts:
- renumbered R38 to R304, R39 to R305, R41 to R306, R40 to R307, R42 to R308, R43 to R309, R45 to R310, R44 to R311, R46 to R312, R47 to R313, R48 to R314, R49 to R315, R34 to R324, R37 to R325, R36 to R326, R35 to R327
Changed lines of the file:
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@@
 		(on_board yes)
 		(dnp no)
-		(property "Reference" "R35"
+		(property "Reference" "R327"
 			(at 151.13 163.83 0)
 			(effects
@@
 			(project "greenenergyecu"
 				(path "/45c1f041-3b7c-4036-abe9-e26621c05a73/5bf5a5f3-cb81-43b4-ad19-7826a949969c"
-					(reference "R35")
+					(reference "R327")
 					(unit 1)
 				)
@@
 		(on_board yes)
 		(dnp no)
-		(property "Reference" "R38"
+		(property "Reference" "R304"
 			(at 151.13 34.29 0)
 			(effects
@@
 			(project "greenenergyecu"
 				(path "/45c1f041-3b7c-4036-abe9-e26621c05a73/5bf5a5f3-cb81-43b4-ad19-7826a949969c"
-					(reference "R38")
+					(reference "R304")
 					(unit 1)
 				)
@@
 		(on_board yes)
 		(dnp no)
-		(property "Reference" "R39"
+		(property "Reference" "R305"
 			(at 153.67 31.75 0)
 			(effects
@@
 			(project "greenenergyecu"
 				(path "/45c1f041-3b7c-4036-abe9-e26621c05a73/5bf5a5f3-cb81-43b4-ad19-7826a949969c"
-					(reference "R39")
+					(reference "R305")
 					(unit 1)
 				)
@@
 		(on_board yes)
 		(dnp no)
-		(property "Reference" "R46"
+		(property "Reference" "R312"
 			(at 151.13 113.03 0)
 			(effects
@@
 			(project "greenenergyecu"
 				(path "/45c1f041-3b7c-4036-abe9-e26621c05a73/5bf5a5f3-cb81-43b4-ad19-7826a949969c"
-					(reference "R46")
+					(reference "R312")
 					(unit 1)
 				)
@@
 		(on_board yes)
 		(dnp no)
-		(property "Reference" "R36"
+		(property "Reference" "R326"
 			(at 148.59 156.21 0)
 			(effects
@@
 			(project "greenenergyecu"
 				(path "/45c1f041-3b7c-4036-abe9-e26621c05a73/5bf5a5f3-cb81-43b4-ad19-7826a949969c"
-					(reference "R36")
+					(reference "R326")
 					(unit 1)
 				)
@@
 		(on_board yes)
 		(dnp no)
-		(property "Reference" "R44"
+		(property "Reference" "R311"
 			(at 153.67 86.36 0)
 			(effects
@@
 			(project "greenenergyecu"
 				(path "/45c1f041-3b7c-4036-abe9-e26621c05a73/5bf5a5f3-cb81-43b4-ad19-7826a949969c"
-					(reference "R44")
+					(reference "R311")
 					(unit 1)
 				)
@@
 		(on_board yes)
 		(dnp no)
-		(property "Reference" "R47"
+		(property "Reference" "R313"
 			(at 153.67 110.49 0)
 			(effects
@@
 			(project "greenenergyecu"
 				(path "/45c1f041-3b7c-4036-abe9-e26621c05a73/5bf5a5f3-cb81-43b4-ad19-7826a949969c"
-					(reference "R47")
+					(reference "R313")
 					(unit 1)
 				)
@@
 		(on_board yes)
 		(dnp no)
-		(property "Reference" "R42"
+		(property "Reference" "R308"
 			(at 151.13 73.66 0)
 			(effects
@@
 			(project "greenenergyecu"
 				(path "/45c1f041-3b7c-4036-abe9-e26621c05a73/5bf5a5f3-cb81-43b4-ad19-7826a949969c"
-					(reference "R42")
+					(reference "R308")
 					(unit 1)
 				)
@@
 		(on_board yes)
 		(dnp no)
-		(property "Reference" "R45"
+		(property "Reference" "R310"
 			(at 151.13 78.74 0)
 			(effects
@@
 			(project "greenenergyecu"
 				(path "/45c1f041-3b7c-4036-abe9-e26621c05a73/5bf5a5f3-cb81-43b4-ad19-7826a949969c"
-					(reference "R45")
+					(reference "R310")
 					(unit 1)
 				)
@@
 		(on_board yes)
 		(dnp no)
-		(property "Reference" "R34"
+		(property "Reference" "R324"
 			(at 148.59 151.13 0)
 			(effects
@@
 			(project "greenenergyecu"
 				(path "/45c1f041-3b7c-4036-abe9-e26621c05a73/5bf5a5f3-cb81-43b4-ad19-7826a949969c"
-					(reference "R34")
+					(reference "R324")
 					(unit 1)
 				)
@@
 		(on_board yes)
 		(dnp no)
-		(property "Reference" "R48"
+		(property "Reference" "R314"
 			(at 151.13 118.11 0)
 			(effects
@@
 			(project "greenenergyecu"
 				(path "/45c1f041-3b7c-4036-abe9-e26621c05a73/5bf5a5f3-cb81-43b4-ad19-7826a949969c"
-					(reference "R48")
+					(reference "R314")
 					(unit 1)
 				)
@@
 		(on_board yes)
 		(dnp no)
-		(property "Reference" "R37"
+		(property "Reference" "R325"
 			(at 152.4 148.59 0)
 			(effects
@@
 			(project "greenenergyecu"
 				(path "/45c1f041-3b7c-4036-abe9-e26621c05a73/5bf5a5f3-cb81-43b4-ad19-7826a949969c"
-					(reference "R37")
+					(reference "R325")
 					(unit 1)
 				)
@@
 		(on_board yes)
 		(dnp no)
-		(property "Reference" "R40"
+		(property "Reference" "R307"
 			(at 153.67 46.99 0)
 			(effects
@@
 			(project "greenenergyecu"
 				(path "/45c1f041-3b7c-4036-abe9-e26621c05a73/5bf5a5f3-cb81-43b4-ad19-7826a949969c"
-					(reference "R40")
+					(reference "R307")
 					(unit 1)
 				)
@@
 		(on_board yes)
 		(dnp no)
-		(property "Reference" "R41"
+		(property "Reference" "R306"
 			(at 151.13 39.37 0)
 			(effects
@@
 			(project "greenenergyecu"
 				(path "/45c1f041-3b7c-4036-abe9-e26621c05a73/5bf5a5f3-cb81-43b4-ad19-7826a949969c"
-					(reference "R41")
+					(reference "R306")
 					(unit 1)
 				)
@@
 		(on_board yes)
 		(dnp no)
-		(property "Reference" "R49"
+		(property "Reference" "R315"
 			(at 153.67 125.73 0)
 			(effects
@@
 			(project "greenenergyecu"
 				(path "/45c1f041-3b7c-4036-abe9-e26621c05a73/5bf5a5f3-cb81-43b4-ad19-7826a949969c"
-					(reference "R49")
+					(reference "R315")
 					(unit 1)
 				)
@@
 		(on_board yes)
 		(dnp no)
-		(property "Reference" "R43"
+		(property "Reference" "R309"
 			(at 153.67 71.12 0)
 			(effects
@@
 			(project "greenenergyecu"
 				(path "/45c1f041-3b7c-4036-abe9-e26621c05a73/5bf5a5f3-cb81-43b4-ad19-7826a949969c"
-					(reference "R43")
-					(unit 1)
-				)
+					(reference "R309")
+					(unit 1)
+				)

Commit message: tilo
Parts:
- removed R304, R306, R308, R310, R312, R314, R324, R326: 4.7k, hellen-one-common:R0603, symbol hellen-one-common:Res
- removed U2, U847, U848, U849: VNLD5160TR-E, Package_SO:SOIC-8_3.9x4.9mm_P1.27mm, symbol chips:VNLD5160
- added G10, G11, G12, G13, G14, G15, G8, G9: PROTO_AREA, footprints:PROTO_AREA1X1, symbol hellen-one-common:PROTO_AREA
- added M9: Module-ign8-0.2, 0.2:ign8, symbol ign8:Module-ign8-0.2
- added Q900, Q901, Q902, Q903, Q904, Q905, Q906, Q907: ISL9V3040D3ST, Package_TO_SOT_SMD:TO-252-2, symbol Device:Q_NIGBT_GCE
- added R900, R901, R902, R903, R904, R905, R906, R907: 22, hellen-one-common:R0603, symbol hellen-one-common:Res
- R305, R307, R309, R311, R313, R315, R325, R327: value 4.7k -> 10k
Connections:
- net GND: now also M9.G (GND), Q900.3 (E), Q901.3 (E), Q902.3 (E), Q903.3 (E), Q904.3 (E), Q905.3 (E), Q906.3 (E), Q907.3 (E)
- net IN1: now also M9.V8 (IGN1)
- net IN2: now also M9.V7 (IGN2)
- net IN3: now also M9.V6 (IGN3)
- net IN4: now also M9.V5 (IGN4)
- net IN5: now also M9.V4 (IGN5)
- net IN6: now also M9.V3 (IGN6)
- net IN7: now also M9.V2 (IGN7)
- net IN8: now also M9.V1 (IGN8)
- net OUT1: now also G8.1, Q900.2 (C)
- net OUT2: now also G9.1, Q901.2 (C)
- net OUT3: now also G10.1, Q902.2 (C)
- net OUT4: now also G11.1, Q903.2 (C)
- net OUT5: now also G12.1, Q904.2 (C)
- net OUT6: now also G13.1, Q905.2 (C)
- net OUT7: now also G14.1, Q906.2 (C)
- net OUT8: now also G15.1, Q907.2 (C)
- new net: Q900.1 (G), R900.1
- new net: Q902.1 (G), R902.1
- new net: M9.S6 (OUT_IGN3), R902.2
- new net: Q901.1 (G), R901.1
- new net: Q906.1 (G), R906.1
- new net: M9.S2 (OUT_IGN7), R906.2
- new net: Q907.1 (G), R907.1
- new net: M9.S1 (OUT_IGN8), R907.2
- new net: M9.S8 (OUT_IGN1), R900.2
- new net: M9.S7 (OUT_IGN2), R901.2
- new net: Q903.1 (G), R903.1
- new net: Q905.1 (G), R905.1
- new net: M9.S3 (OUT_IGN6), R905.2
- new net: Q904.1 (G), R904.1
- new net: M9.S4 (OUT_IGN5), R904.2
- new net: M9.S5 (OUT_IGN4), R903.2
- new net 33v: M9.V10 (V33)
- new net 5v: M9.V9 (VCC)
- no-connect marks 8 -> 0
Other:
- moved on the sheet: R305, R307, R309, R311, R313, R315, R325, R327

Commit message: tilo
Parts:
- R305, R307, R309, R311, R313, R315, R325, R327: LCSC C23162 -> C17414
Changed lines of the file:
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@@
 			)
 		)
-		(property "LCSC" "C23162"
+		(property "LCSC" "C17414"
 			(at 271.78 152.4 0)
 			(effects
@@
 			)
 		)
-		(property "LCSC" "C23162"
+		(property "LCSC" "C17414 "
 			(at 274.32 30.48 0)
 			(effects
@@
 			)
 		)
-		(property "LCSC" "C23162"
+		(property "LCSC" "C17414"
 			(at 274.32 74.93 0)
 			(effects
@@
 			)
 		)
-		(property "LCSC" "C23162"
+		(property "LCSC" "C17414"
 			(at 274.32 109.22 0)
 			(effects
@@
 			)
 		)
-		(property "LCSC" "C23162"
+		(property "LCSC" "C17414"
 			(at 273.05 147.32 0)
 			(effects
@@
 			)
 		)
-		(property "LCSC" "C23162"
+		(property "LCSC" "C17414"
 			(at 274.32 35.56 0)
 			(effects
@@
 			)
 		)
-		(property "LCSC" "C23162"
+		(property "LCSC" "C17414"
 			(at 274.32 114.3 0)
 			(effects
@@
 			)
 		)
-		(property "LCSC" "C23162"
+		(property "LCSC" "C17414"
 			(at 274.32 69.85 0)
 			(effects

Commit message: tilo
Parts:
- R305: LCSC C17414 -> C17414
Changed lines of the file:
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@@
 			)
 		)
-		(property "LCSC" "C17414 "
+		(property "LCSC" "C17414"
 			(at 274.32 30.48 0)
 			(effects

Commit message: casi
Connections:
- net IN7: now also M9.V1 (IGN8), R327.1; no longer M9.V2 (IGN7), R325.1
- net IN8: now also M9.V2 (IGN7), R325.1; no longer M9.V1 (IGN8), R327.1
Changed lines of the file:
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@@
 		)
 	)
-	(hierarchical_label "IN7"
+	(hierarchical_label "IN8"
 		(shape input)
 		(at 274.32 147.32 0)
@@
 		)
 	)
-	(hierarchical_label "IN8"
+	(hierarchical_label "IN7"
 		(shape input)
 		(at 273.05 152.4 0)

Commit message: holi
Parts:
- Q900, Q901, Q902, Q903, Q904, Q905, Q906, Q907: LCSC (none) -> C903784; MyComment DNP -> (none)
Changed lines of the file:
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@@
 			)
 		)
-		(property "LCSC" ""
+		(property "LCSC" "C903784"
 			(at 54.61 34.29 0)
 			(effects
@@
 			)
 		)
-		(property "MyComment" "DNP"
+		(property "MyComment" ""
 			(at 57.15 37.592 0)
 			(effects
@@
 			)
 		)
-		(property "LCSC" ""
+		(property "LCSC" "C903784"
 			(at 49.53 73.66 0)
 			(effects
@@
 			)
 		)
-		(property "MyComment" "DNP"
+		(property "MyComment" ""
 			(at 52.07 76.962 0)
 			(effects
@@
 			)
 		)
-		(property "LCSC" ""
+		(property "LCSC" "C903784"
 			(at 81.28 41.91 0)
 			(effects
@@
 			)
 		)
-		(property "MyComment" "DNP"
+		(property "MyComment" ""
 			(at 83.82 45.212 0)
 			(effects
@@
 			)
 		)
-		(property "LCSC" ""
+		(property "LCSC" "C903784"
 			(at 76.2 81.28 0)
 			(effects
@@
 			)
 		)
-		(property "MyComment" "DNP"
+		(property "MyComment" ""
 			(at 78.74 84.582 0)
 			(effects
@@
 			)
 		)
-		(property "LCSC" ""
+		(property "LCSC" "C903784"
 			(at 44.45 151.13 0)
 			(effects
@@
 			)
 		)
-		(property "MyComment" "DNP"
+		(property "MyComment" ""
 			(at 46.99 154.432 0)
 			(effects
@@
 					(size 1.27 1.27)
 				)
+				(hide yes)
 			)
 		)
@@
 			)
 		)
-		(property "LCSC" ""
+		(property "LCSC" "C903784"
 			(at 76.2 120.65 0)
 			(effects
@@
 			)
 		)
-		(property "MyComment" "DNP"
+		(property "MyComment" ""
 			(at 78.74 123.952 0)
 			(effects
@@
 			)
 		)
-		(property "LCSC" ""
+		(property "LCSC" "C903784"
 			(at 49.53 113.03 0)
 			(effects
@@
 			)
 		)
-		(property "MyComment" "DNP"
+		(property "MyComment" ""
 			(at 52.07 116.332 0)
 			(effects
@@
 					(size 1.27 1.27)
 				)
+				(hide yes)
 			)
 		)
@@
 			)
 		)
-		(property "LCSC" ""
+		(property "LCSC" "C903784"
 			(at 71.12 158.75 0)
 			(effects
@@
 			)
 		)
-		(property "MyComment" "DNP"
+		(property "MyComment" ""
 			(at 73.66 162.052 0)
 			(effects
@@
 					(size 1.27 1.27)
 				)
+				(hide yes)
 			)
 		)

Commit message: ww
Parts:
- removed G10, G11, G12, G13, G14, G15, G8, G9: PROTO_AREA, footprints:PROTO_AREA1X1, symbol hellen-one-common:PROTO_AREA
