File: INJ6.kicad_sch (KiCad schematic)
At the start: 25 parts, among them M9 Module-ign8-0.2, Q900 ISL9V3040D3ST, Q901 ISL9V3040D3ST, Q902 ISL9V3040D3ST, Q903 ISL9V3040D3ST, Q904 ISL9V3040D3ST, Q905 ISL9V3040D3ST, Q906 ISL9V3040D3ST, Q907 ISL9V3040D3ST

Commit message: wew
Parts:
- Q900, Q901, Q902, Q903, Q904, Q905, Q906, Q907: LCSC C903784 -> C5350881
Changed lines of the file:
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@@
 			)
 		)
-		(property "LCSC" "C903784"
+		(property "LCSC" "C5350881"
 			(at 54.61 34.29 0)
 			(effects
@@
 			)
 		)
-		(property "LCSC" "C903784"
+		(property "LCSC" "C5350881"
 			(at 49.53 73.66 0)
 			(effects
@@
 			)
 		)
-		(property "LCSC" "C903784"
+		(property "LCSC" "C5350881"
 			(at 81.28 41.91 0)
 			(effects
@@
 			)
 		)
-		(property "LCSC" "C903784"
+		(property "LCSC" "C5350881"
 			(at 76.2 81.28 0)
 			(effects
@@
 			)
 		)
-		(property "LCSC" "C903784"
+		(property "LCSC" "C5350881"
 			(at 44.45 151.13 0)
 			(effects
@@
 			)
 		)
-		(property "LCSC" "C903784"
+		(property "LCSC" "C5350881"
 			(at 76.2 120.65 0)
 			(effects
@@
 			)
 		)
-		(property "LCSC" "C903784"
+		(property "LCSC" "C5350881"
 			(at 49.53 113.03 0)
 			(effects
@@
 			)
 		)
-		(property "LCSC" "C903784"
+		(property "LCSC" "C5350881"
 			(at 71.12 158.75 0)
 			(effects

Commit message: a
Parts:
- Q901: footprint Package_TO_SOT_SMD:TO-252-2 -> hellen-one-common:abel-252-2
Changed lines of the file:
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@@
 			)
 		)
-		(property "Footprint" "Package_TO_SOT_SMD:TO-252-2"
+		(property "Footprint" "hellen-one-common:abel-252-2"
 			(at 76.2 39.37 0)
 			(effects
