File: IGN6.kicad_sch (KiCad schematic)
At the start: 24 parts, among them Q1 ISL9V3040D3ST, Q2 ISL9V3040D3ST, Q3 ISL9V3040D3ST, Q4 ISL9V3040D3ST, Q5 ISL9V3040D3ST, Q6 ISL9V3040D3ST

Commit message: weW
Parts:
- renumbered F9 to F10, F4 to F5, F5 to F6, F6 to F7, F7 to F8, F8 to F9
Changed lines of the file:
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@@
 		(on_board yes)
 		(dnp no)
-		(property "Reference" "F7"
+		(property "Reference" "F8"
 			(at 181.61 64.77 90)
 			(effects
@@
 			(project "greenenergyecu"
 				(path "/45c1f041-3b7c-4036-abe9-e26621c05a73/f08b5b09-fcb6-4f5b-8ff2-a721d01c34bf"
-					(reference "F7")
+					(reference "F8")
 					(unit 1)
 				)
@@
 		(on_board yes)
 		(dnp no)
-		(property "Reference" "F9"
+		(property "Reference" "F10"
 			(at 181.61 120.65 90)
 			(effects
@@
 			(project "greenenergyecu"
 				(path "/45c1f041-3b7c-4036-abe9-e26621c05a73/f08b5b09-fcb6-4f5b-8ff2-a721d01c34bf"
-					(reference "F9")
+					(reference "F10")
 					(unit 1)
 				)
@@
 		(on_board yes)
 		(dnp no)
-		(property "Reference" "F5"
+		(property "Reference" "F6"
 			(at 134.62 92.71 90)
 			(effects
@@
 			(project "greenenergyecu"
 				(path "/45c1f041-3b7c-4036-abe9-e26621c05a73/f08b5b09-fcb6-4f5b-8ff2-a721d01c34bf"
-					(reference "F5")
+					(reference "F6")
 					(unit 1)
 				)
@@
 		(on_board yes)
 		(dnp no)
-		(property "Reference" "F6"
+		(property "Reference" "F7"
 			(at 134.62 120.65 90)
 			(effects
@@
 			(project "greenenergyecu"
 				(path "/45c1f041-3b7c-4036-abe9-e26621c05a73/f08b5b09-fcb6-4f5b-8ff2-a721d01c34bf"
-					(reference "F6")
+					(reference "F7")
 					(unit 1)
 				)
@@
 		(on_board yes)
 		(dnp no)
-		(property "Reference" "F8"
+		(property "Reference" "F9"
 			(at 181.61 92.71 90)
 			(effects
@@
 			(project "greenenergyecu"
 				(path "/45c1f041-3b7c-4036-abe9-e26621c05a73/f08b5b09-fcb6-4f5b-8ff2-a721d01c34bf"
-					(reference "F8")
+					(reference "F9")
 					(unit 1)
 				)
@@
 		(on_board yes)
 		(dnp no)
-		(property "Reference" "F4"
+		(property "Reference" "F5"
 			(at 134.62 64.77 90)
 			(effects
@@
 			(project "greenenergyecu"
 				(path "/45c1f041-3b7c-4036-abe9-e26621c05a73/f08b5b09-fcb6-4f5b-8ff2-a721d01c34bf"
-					(reference "F4")
-					(unit 1)
-				)
+					(reference "F5")
+					(unit 1)
+				)

Commit message: weW
Parts:
- renumbered F5 to F844, F6 to F845, F7 to F846, F8 to F847, F9 to F848, F10 to F849, Q1 to Q841, Q2 to Q842, Q3 to Q843, Q4 to Q844, Q5 to Q845, Q6 to Q846, R22 to R867, R23 to R868, R24 to R869, R25 to R870, R26 to R871, R27 to R872, R28 to R873, R29 to R874, R30 to R875, R31 to R876, R32 to R877, R33 to R878
Changed lines of the file:
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@@
 		(on_board yes)
 		(dnp no)
-		(property "Reference" "R32"
+		(property "Reference" "R877"
 			(at 172.3996 87.5253 0)
 			(effects
@@
 			(project "greenenergyecu"
 				(path "/45c1f041-3b7c-4036-abe9-e26621c05a73/f08b5b09-fcb6-4f5b-8ff2-a721d01c34bf"
-					(reference "R32")
+					(reference "R877")
 					(unit 1)
 				)
@@
 		(on_board yes)
 		(dnp no)
-		(property "Reference" "R29"
+		(property "Reference" "R874"
 			(at 172.962 92.9018 0)
 			(effects
@@
 			(project "greenenergyecu"
 				(path "/45c1f041-3b7c-4036-abe9-e26621c05a73/f08b5b09-fcb6-4f5b-8ff2-a721d01c34bf"
-					(reference "R29")
+					(reference "R874")
 					(unit 1)
 				)
@@
 		(on_board yes)
 		(dnp no)
-		(property "Reference" "R31"
+		(property "Reference" "R876"
 			(at 172.3996 59.5853 0)
 			(effects
@@
 			(project "greenenergyecu"
 				(path "/45c1f041-3b7c-4036-abe9-e26621c05a73/f08b5b09-fcb6-4f5b-8ff2-a721d01c34bf"
-					(reference "R31")
+					(reference "R876")
 					(unit 1)
 				)
@@
 		(on_board yes)
 		(dnp no)
-		(property "Reference" "R33"
+		(property "Reference" "R878"
 			(at 172.3996 115.4653 0)
 			(effects
@@
 			(project "greenenergyecu"
 				(path "/45c1f041-3b7c-4036-abe9-e26621c05a73/f08b5b09-fcb6-4f5b-8ff2-a721d01c34bf"
-					(reference "R33")
+					(reference "R878")
 					(unit 1)
 				)
@@
 		(on_board yes)
 		(dnp no)
-		(property "Reference" "R26"
+		(property "Reference" "R871"
 			(at 125.4096 87.5253 0)
 			(effects
@@
 			(project "greenenergyecu"
 				(path "/45c1f041-3b7c-4036-abe9-e26621c05a73/f08b5b09-fcb6-4f5b-8ff2-a721d01c34bf"
-					(reference "R26")
+					(reference "R871")
 					(unit 1)
 				)
@@
 		(on_board yes)
 		(dnp no)
-		(property "Reference" "R25"
+		(property "Reference" "R870"
 			(at 125.4096 59.5853 0)
 			(effects
@@
 			(project "greenenergyecu"
 				(path "/45c1f041-3b7c-4036-abe9-e26621c05a73/f08b5b09-fcb6-4f5b-8ff2-a721d01c34bf"
-					(reference "R25")
+					(reference "R870")
 					(unit 1)
 				)
@@
 		(on_board yes)
 		(dnp no)
-		(property "Reference" "R27"
+		(property "Reference" "R872"
 			(at 125.4096 115.4653 0)
 			(effects
@@
 			(project "greenenergyecu"
 				(path "/45c1f041-3b7c-4036-abe9-e26621c05a73/f08b5b09-fcb6-4f5b-8ff2-a721d01c34bf"
-					(reference "R27")
+					(reference "R872")
 					(unit 1)
 				)
@@
 		(on_board yes)
 		(dnp no)
-		(property "Reference" "Q6"
+		(property "Reference" "Q846"
 			(at 157.7086 122.0216 0)
 			(effects
@@
 			(project "greenenergyecu"
 				(path "/45c1f041-3b7c-4036-abe9-e26621c05a73/f08b5b09-fcb6-4f5b-8ff2-a721d01c34bf"
-					(reference "Q6")
+					(reference "Q846")
 					(unit 1)
 				)
@@
 		(on_board yes)
 		(dnp no)
-		(property "Reference" "R28"
+		(property "Reference" "R873"
 			(at 172.962 64.9618 0)
 			(effects
@@
 			(project "greenenergyecu"
 				(path "/45c1f041-3b7c-4036-abe9-e26621c05a73/f08b5b09-fcb6-4f5b-8ff2-a721d01c34bf"
-					(reference "R28")
+					(reference "R873")
 					(unit 1)
 				)
@@
 		(on_board yes)
 		(dnp no)
-		(property "Reference" "Q4"
+		(property "Reference" "Q844"
 			(at 157.7086 66.1416 0)
 			(effects
@@
 			(project "greenenergyecu"
 				(path "/45c1f041-3b7c-4036-abe9-e26621c05a73/f08b5b09-fcb6-4f5b-8ff2-a721d01c34bf"
-					(reference "Q4")
+					(reference "Q844")
 					(unit 1)
 				)
@@
 		(on_board yes)
 		(dnp no)
-		(property "Reference" "F8"
+		(property "Reference" "F847"
 			(at 181.61 64.77 90)
 			(effects
@@
 			(project "greenenergyecu"
 				(path "/45c1f041-3b7c-4036-abe9-e26621c05a73/f08b5b09-fcb6-4f5b-8ff2-a721d01c34bf"
-					(reference "F8")
+					(reference "F847")
 					(unit 1)
 				)
@@
 		(on_board yes)
 		(dnp no)
-		(property "Reference" "F10"
+		(property "Reference" "F849"
 			(at 181.61 120.65 90)
 			(effects
@@
 			(project "greenenergyecu"
 				(path "/45c1f041-3b7c-4036-abe9-e26621c05a73/f08b5b09-fcb6-4f5b-8ff2-a721d01c34bf"
-					(reference "F10")
+					(reference "F849")
 					(unit 1)
 				)
@@
 		(on_board yes)
 		(dnp no)
-		(property "Reference" "Q2"
+		(property "Reference" "Q842"
 			(at 110.7186 94.0816 0)
 			(effects
@@
 			(project "greenenergyecu"
 				(path "/45c1f041-3b7c-4036-abe9-e26621c05a73/f08b5b09-fcb6-4f5b-8ff2-a721d01c34bf"
-					(reference "Q2")
+					(reference "Q842")
 					(unit 1)
 				)
@@
 		(on_board yes)
 		(dnp no)
-		(property "Reference" "Q5"
+		(property "Reference" "Q845"
 			(at 157.7086 94.0816 0)
 			(effects
@@
 			(project "greenenergyecu"
 				(path "/45c1f041-3b7c-4036-abe9-e26621c05a73/f08b5b09-fcb6-4f5b-8ff2-a721d01c34bf"
-					(reference "Q5")
+					(reference "Q845")
 					(unit 1)
 				)
@@
 		(on_board yes)
 		(dnp no)
-		(property "Reference" "R30"
+		(property "Reference" "R875"
 			(at 172.962 120.8418 0)
 			(effects
@@
 			(project "greenenergyecu"
 				(path "/45c1f041-3b7c-4036-abe9-e26621c05a73/f08b5b09-fcb6-4f5b-8ff2-a721d01c34bf"
-					(reference "R30")
+					(reference "R875")
 					(unit 1)
 				)
@@
 		(on_board yes)
 		(dnp no)
-		(property "Reference" "R22"
+		(property "Reference" "R867"
 			(at 125.972 64.9618 0)
 			(effects
@@
 			(project "greenenergyecu"
 				(path "/45c1f041-3b7c-4036-abe9-e26621c05a73/f08b5b09-fcb6-4f5b-8ff2-a721d01c34bf"
-					(reference "R22")
+					(reference "R867")
 					(unit 1)
 				)
@@
 		(on_board yes)
 		(dnp no)
-		(property "Reference" "F6"
+		(property "Reference" "F845"
 			(at 134.62 92.71 90)
 			(effects
@@
 			(project "greenenergyecu"
 				(path "/45c1f041-3b7c-4036-abe9-e26621c05a73/f08b5b09-fcb6-4f5b-8ff2-a721d01c34bf"
-					(reference "F6")
+					(reference "F845")
 					(unit 1)
 				)
@@
 		(on_board yes)
 		(dnp no)
-		(property "Reference" "Q1"
+		(property "Reference" "Q841"
 			(at 110.7186 66.1416 0)
 			(effects
@@
 			(project "greenenergyecu"
 				(path "/45c1f041-3b7c-4036-abe9-e26621c05a73/f08b5b09-fcb6-4f5b-8ff2-a721d01c34bf"
-					(reference "Q1")
+					(reference "Q841")
 					(unit 1)
 				)
@@
 		(on_board yes)
 		(dnp no)
-		(property "Reference" "F7"
+		(property "Reference" "F846"
 			(at 134.62 120.65 90)
 			(effects
@@
 			(project "greenenergyecu"
 				(path "/45c1f041-3b7c-4036-abe9-e26621c05a73/f08b5b09-fcb6-4f5b-8ff2-a721d01c34bf"
-					(reference "F7")
+					(reference "F846")
 					(unit 1)
 				)
@@
 		(on_board yes)
 		(dnp no)
-		(property "Reference" "R23"
+		(property "Reference" "R868"
 			(at 125.972 92.9018 0)
 			(effects
@@
 			(project "greenenergyecu"
 				(path "/45c1f041-3b7c-4036-abe9-e26621c05a73/f08b5b09-fcb6-4f5b-8ff2-a721d01c34bf"
-					(reference "R23")
+					(reference "R868")
 					(unit 1)
 				)
@@
 		(on_board yes)
 		(dnp no)
-		(property "Reference" "F9"
+		(property "Reference" "F848"
 			(at 181.61 92.71 90)
 			(effects
@@
 			(project "greenenergyecu"
 				(path "/45c1f041-3b7c-4036-abe9-e26621c05a73/f08b5b09-fcb6-4f5b-8ff2-a721d01c34bf"
-					(reference "F9")
+					(reference "F848")
 					(unit 1)
 				)
@@
 		(on_board yes)
 		(dnp no)
-		(property "Reference" "Q3"
+		(property "Reference" "Q843"
 			(at 110.7186 122.0216 0)
 			(effects
@@
 			(project "greenenergyecu"
 				(path "/45c1f041-3b7c-4036-abe9-e26621c05a73/f08b5b09-fcb6-4f5b-8ff2-a721d01c34bf"
-					(reference "Q3")
+					(reference "Q843")
 					(unit 1)
 				)
@@
 		(on_board yes)
 		(dnp no)
-		(property "Reference" "R24"
+		(property "Reference" "R869"
 			(at 125.972 120.8418 0)
 			(effects
@@
 			(project "greenenergyecu"
 				(path "/45c1f041-3b7c-4036-abe9-e26621c05a73/f08b5b09-fcb6-4f5b-8ff2-a721d01c34bf"
-					(reference "R24")
+					(reference "R869")
 					(unit 1)
 				)
@@
 		(on_board yes)
 		(dnp no)
-		(property "Reference" "F5"
+		(property "Reference" "F844"
 			(at 134.62 64.77 90)
 			(effects
@@
 			(project "greenenergyecu"
 				(path "/45c1f041-3b7c-4036-abe9-e26621c05a73/f08b5b09-fcb6-4f5b-8ff2-a721d01c34bf"
-					(reference "F5")
-					(unit 1)
-				)
+					(reference "F844")
+					(unit 1)
+				)

Commit message: tilo
Parts:
- added F850, F851: 50mA, Fuse:Fuse_0603_1608Metric, symbol Device:Polyfuse
- added G1, G16, G2, G3, G4, G5, G6, G7: PROTO_AREA, footprints:PROTO_AREA1X1, symbol hellen-one-common:PROTO_AREA
- added Q847, Q849: ISL9V3040D3ST, Package_TO_SOT_SMD:TO-252-2, symbol Device:Q_NIGBT_GCE
- added R700, R701: 22, hellen-one-common:R0603, symbol hellen-one-common:Res
- added R879, R880: 0, Resistor_SMD:R_2512_6332Metric, symbol hellen-one-common:Res
Connections:
- net GND: now also Q847.3 (E), Q849.3 (E)
- net OUT1: now also G2.1
- net OUT2: now also G3.1
- net OUT3: now also G4.1
- net OUT4: now also G5.1
- net OUT5: now also G6.1
- net OUT6: now also G7.1
- new net: F850.1, R700.2, R879.1
- new net: Q849.1 (G), R701.1
- new net: Q847.1 (G), R700.1
- new net: F851.1, R701.2, R880.1
- new net IN7: F850.2
- new net IN8: F851.2
- new net OUT7: G1.1, Q847.2 (C), R879.2
- new net OUT8: G16.1, Q849.2 (C), R880.2

Commit message: w
Parts:
- Q841, Q842, Q843, Q844, Q845, Q846, Q847, Q849: LCSC (none) -> C903784; MyComment DNP -> (none)
- R870, R871, R872, R876, R877, R878, R879: LCSC C25469 -> (none); comentario (none) -> DNP
- R880: LCSC C25469 -> (none); MyComment (none) -> DNP
Changed lines of the file:
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@@
 			)
 		)
-		(property "LCSC" "C25469"
+		(property "LCSC" ""
 			(at 177.8 90.17 0)
 			(effects
@@
 			)
 		)
-		(property "comentario" ""
+		(property "comentario" "DNP"
 			(at 177.8 90.17 0)
 			(effects
@@
 			)
 		)
-		(property "LCSC" "C25469"
+		(property "LCSC" ""
 			(at 177.8 62.23 0)
 			(effects
@@
 			)
 		)
-		(property "comentario" ""
+		(property "comentario" "DNP"
 			(at 177.8 62.23 0)
 			(effects
@@
 					(size 1.27 1.27)
 				)
-				(hide yes)
 			)
 		)
@@
 			)
 		)
-		(property "LCSC" "C25469"
+		(property "LCSC" ""
 			(at 177.8 118.11 0)
 			(effects
@@
 			)
 		)
-		(property "comentario" ""
+		(property "comentario" "DNP"
 			(at 177.8 118.11 0)
 			(effects
@@
 			)
 		)
-		(property "LCSC" ""
+		(property "LCSC" "C903784"
 			(at 163.83 154.94 0)
 			(effects
@@
 			)
 		)
-		(property "MyComment" "DNP"
+		(property "MyComment" ""
 			(at 165.354 161.036 0)
 			(effects
@@
 			)
 		)
-		(property "LCSC" "C25469"
+		(property "LCSC" ""
 			(at 130.81 90.17 0)
 			(effects
@@
 			)
 		)
-		(property "comentario" ""
+		(property "comentario" "DNP"
 			(at 130.81 90.17 0)
 			(effects
@@
 					(size 1.27 1.27)
 				)
-				(hide yes)
 			)
 		)
@@
 			)
 		)
-		(property "LCSC" "C25469"
+		(property "LCSC" ""
 			(at 130.81 62.23 0)
 			(effects
@@
 			)
 		)
-		(property "comentario" ""
+		(property "comentario" "DNP"
 			(at 130.81 62.23 0)
 			(effects
@@
 					(size 1.27 1.27)
 				)
-				(hide yes)
 			)
 		)
@@
 			)
 		)
-		(property "LCSC" "C25469"
+		(property "LCSC" ""
 			(at 130.81 118.11 0)
 			(effects
@@
 			)
 		)
-		(property "comentario" ""
+		(property "comentario" "DNP"
 			(at 130.81 118.11 0)
 			(effects
@@
 			)
 		)
-		(property "LCSC" "C25469"
+		(property "LCSC" ""
 			(at 132.08 149.86 0)
 			(effects
@@
 			)
 		)
-		(property "comentario" ""
+		(property "comentario" "DNP"
 			(at 132.08 149.86 0)
 			(effects
@@
 			)
 		)
-		(property "LCSC" ""
+		(property "LCSC" "C903784"
 			(at 116.84 154.94 0)
 			(effects
@@
 			)
 		)
-		(property "MyComment" "DNP"
+		(property "MyComment" ""
 			(at 110.49 158.75 0)
 			(effects
@@
 			)
 		)
-		(property "LCSC" ""
+		(property "LCSC" "C903784"
 			(at 162.56 123.19 0)
 			(effects
@@
 			)
 		)
-		(property "MyComment" "DNP"
+		(property "MyComment" ""
 			(at 164.084 129.286 0)
 			(effects
@@
 			)
 		)
-		(property "LCSC" ""
+		(property "LCSC" "C903784"
 			(at 162.56 67.31 0)
 			(effects
@@
 			)
 		)
-		(property "MyComment" "DNP"
+		(property "MyComment" ""
 			(at 156.21 71.12 0)
 			(effects
@@
 			)
 		)
-		(property "LCSC" ""
+		(property "LCSC" "C903784"
 			(at 115.57 95.25 0)
 			(effects
@@
 			)
 		)
-		(property "MyComment" "DNP"
+		(property "MyComment" ""
 			(at 109.22 99.06 0)
 			(effects
@@
 			)
 		)
-		(property "LCSC" ""
+		(property "LCSC" "C903784"
 			(at 162.56 95.25 0)
 			(effects
@@
 			)
 		)
-		(property "MyComment" "DNP"
+		(property "MyComment" ""
 			(at 156.21 99.06 0)
 			(effects
@@
 			)
 		)
-		(property "LCSC" ""
+		(property "LCSC" "C903784"
 			(at 115.57 67.31 0)
 			(effects
@@
 			)
 		)
-		(property "MyComment" "DNP"
+		(property "MyComment" ""
 			(at 118.11 70.612 0)
 			(effects
@@
 			)
 		)
-		(property "LCSC" "C25469"
+		(property "LCSC" ""
 			(at 179.07 149.86 0)
 			(effects
@@
 			)
 		)
-		(property "comentario" ""
+		(property "MyComment" "DNP"
 			(at 179.07 149.86 0)
 			(effects
@@
 					(size 1.27 1.27)
 				)
-				(hide yes)
 			)
 		)
@@
 			)
 		)
-		(property "LCSC" ""
+		(property "LCSC" "C903784"
 			(at 115.57 123.19 0)
 			(effects
@@
 			)
 		)
-		(property "MyComment" "DNP"
+		(property "MyComment" ""
 			(at 109.22 127 0)
 			(effects

Commit message: ww
Changed lines of the file:
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@@
 					(size 1.27 1.27)
 				)
-				(hide yes)
 			)
 		)
@@
 					(size 1.27 1.27)
 				)
-				(hide yes)
 			)
 		)
@@
 					(size 1.27 1.27)
 				)
-				(hide yes)
 			)
 		)
@@
 					(size 1.27 1.27)
 				)
-				(hide yes)
-			)
-		)
+			)
+		)

Commit message: ww
Parts:
- removed G1, G16, G2, G3, G4, G5, G6, G7: PROTO_AREA, footprints:PROTO_AREA1X1, symbol hellen-one-common:PROTO_AREA

Commit message: wew
Parts:
- Q841, Q842, Q843, Q844, Q845, Q846, Q847, Q849: LCSC C903784 -> C462128
Changed lines of the file:
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@@
 			)
 		)
-		(property "LCSC" "C903784"
+		(property "LCSC" "C462128"
 			(at 163.83 154.94 0)
 			(effects
@@
 			)
 		)
-		(property "LCSC" "C903784"
+		(property "LCSC" "C462128"
 			(at 116.84 154.94 0)
 			(effects
@@
 			)
 		)
-		(property "LCSC" "C903784"
+		(property "LCSC" "C462128"
 			(at 162.56 123.19 0)
 			(effects
@@
 			)
 		)
-		(property "LCSC" "C903784"
+		(property "LCSC" "C462128"
 			(at 162.56 67.31 0)
 			(effects
@@
 			)
 		)
-		(property "LCSC" "C903784"
+		(property "LCSC" "C462128"
 			(at 115.57 95.25 0)
 			(effects
@@
 			)
 		)
-		(property "LCSC" "C903784"
+		(property "LCSC" "C462128"
 			(at 162.56 95.25 0)
 			(effects
@@
 			)
 		)
-		(property "LCSC" "C903784"
+		(property "LCSC" "C462128"
 			(at 115.57 67.31 0)
 			(effects
@@
 			)
 		)
-		(property "LCSC" "C903784"
+		(property "LCSC" "C462128"
 			(at 115.57 123.19 0)
 			(effects

Commit message: wew
Parts:
- Q846, Q847, Q849: footprint Package_TO_SOT_SMD:TO-252-2 -> hellen-one-common:TO-252-2MODD
Changed lines of the file:
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@@
 			)
 		)
-		(property "Footprint" "Package_TO_SOT_SMD:TO-252-2"
+		(property "Footprint" "hellen-one-common:TO-252-2MODD"
 			(at 158.75 152.4 0)
 			(effects
@@
 			)
 		)
-		(property "Footprint" "Package_TO_SOT_SMD:TO-252-2"
+		(property "Footprint" "hellen-one-common:TO-252-2MODD"
 			(at 111.76 152.4 0)
 			(effects
@@
 			)
 		)
-		(property "Footprint" "Package_TO_SOT_SMD:TO-252-2"
+		(property "Footprint" "hellen-one-common:TO-252-2MODD"
 			(at 157.48 120.65 0)
 			(effects
