File: IGN6.kicad_sch (KiCad schematic)
At the start: 32 parts, among them Q841 ISL9V3040D3ST, Q842 ISL9V3040D3ST, Q843 ISL9V3040D3ST, Q844 ISL9V3040D3ST, Q845 ISL9V3040D3ST, Q846 ISL9V3040D3ST, Q847 ISL9V3040D3ST, Q849 ISL9V3040D3ST

Commit message: w
Parts:
- Q845: footprint hellen-one-common:TO-252-2MODD -> hellen-one-common:MODIGBT
Changed lines of the file:
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@@
 			)
 		)
-		(property "Footprint" "hellen-one-common:TO-252-2MODD"
+		(property "Footprint" "hellen-one-common:MODIGBT"
 			(at 157.48 92.71 0)
 			(effects
