File: IGN6.kicad_sch (KiCad schematic)
At the start: 32 parts, among them Q841 ISL9V3040D3ST, Q842 ISL9V3040D3ST, Q843 ISL9V3040D3ST, Q844 ISL9V3040D3ST, Q845 ISL9V3040D3ST, Q846 ISL9V3040D3ST, Q847 ISL9V3040D3ST, Q849 ISL9V3040D3ST

Commit message: w
Parts:
- Q842, Q843, Q849: footprint Package_TO_SOT_SMD:TO-252-2 -> hellen-one-common:MODIGBT
Changed lines of the file:
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@@
 			)
 		)
-		(property "Footprint" "Package_TO_SOT_SMD:TO-252-2"
+		(property "Footprint" "hellen-one-common:MODIGBT"
 			(at 158.75 152.4 0)
 			(effects
@@
 			)
 		)
-		(property "Footprint" "Package_TO_SOT_SMD:TO-252-2"
+		(property "Footprint" "hellen-one-common:MODIGBT"
 			(at 110.49 92.71 0)
 			(effects
@@
 			)
 		)
-		(property "Footprint" "Package_TO_SOT_SMD:TO-252-2"
+		(property "Footprint" "hellen-one-common:MODIGBT"
 			(at 110.49 120.65 0)
 			(effects
